File: RF_INPUT_BREAKOUT/RF_INPUT_BREAKOUT-backups/RF_INPUT_BREAKOUT-2025-09-19_165512/RF_INPUT_BREAKOUT.kicad_pcb (KiCad board)
At the start: 4 copper layers, 121 x 65 mm, 26 parts, among them IC1 SI4705-D62-GM, J5 Conn_2Rows-21Pins, U1 LD1117S33TR_SOT223, U2 LT5512EUF-PBF, X1 ASE-xxxMHz

Commit message: redid layout
Parts:
- removed R10, R7, R8, R9: 330, Resistor_SMD:R_0402_1005Metric
- added R1: 4.7k, Resistor_SMD:R_0402_1005Metric, F.Cu at (123.5, 91.0)
- added R2: 4.7k, Resistor_SMD:R_0402_1005Metric, F.Cu at (127.0, 91.5)
- moved L1 264.4 mm to (-36.1, -7.51), turned to 0 degrees
- moved L2 263.4 mm to (-36.1, -6.01), turned to 0 degrees
- moved C1 33.1 mm to (116.0, 70.0), turned to 0 degrees
- moved C2 27.7 mm to (123.5, 72.8), turned to 90 degrees
- moved U1 27.5 mm to (114.3, 75.2), turned to 180 degrees
- moved C9 18.6 mm to (112.0, 87.5), turned to -90 degrees
- moved C5 16.5 mm to (118.0, 80.0), turned to 180 degrees
- moved R6 13.8 mm to (116.6, 91.0), turned to 180 degrees
- moved R3 13.5 mm to (118.0, 81.5), turned to 0 degrees
- moved X1 13.2 mm to (106.0, 88.5)
- moved C8 11.8 mm to (118.6, 92.0), turned to 0 degrees
- moved C6 11.3 mm to (116.0, 83.0), turned to 180 degrees
- moved C7 11.1 mm to (118.6, 91.0), turned to 0 degrees
- moved U2 10.5 mm to (118.0, 87.5), turned to 0 degrees
- moved R4 9.11 mm to (127.5, 99.0), turned to 0 degrees
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Connections:
- IC1 pad 8: /MCU_I2S_SDIO -> /MCU_I2C_SCLK
- J5 pad 1: GND -> +5V
- J5 pad 11: /RF_ANALOG_ROUT -> /RF_ANALOG_LOUT
- J5 pad 13: /MCU_RF_RCLK -> /RF_ANALOG_ROUT
- J5 pad 15: Net-(J5-Pin_15) -> /MCU_I2C_SCLK
- J5 pad 17: Net-(J5-Pin_17) -> /MCU_I2C_SCLK
- J5 pad 19: Net-(J5-Pin_19) -> /MCU_RF_SEN
- J5 pad 21: Net-(J5-Pin_21) -> /MCU_RF_RST
- J5 pad 3: /RF_I2S_DCLK -> GND
- J5 pad 5: /RF_I2S_DFS -> /RF_I2S_DCLK
- J5 pad 7: /RF_I2S_DOUT -> /RF_I2S_DFS
- J5 pad 9: /RF_ANALOG_LOUT -> /RF_I2S_DOUT
Routing:
- net Net-(J5-Pin_21): track 12.6 -> 0.00 mm
- net Net-(J5-Pin_19): track 10.7 -> 0.00 mm
- net Net-(J5-Pin_17): track 8.86 -> 0.00 mm
- net /MCU_RF_RCLK: track 8.80 -> 0.00 mm
- net +3.3V: track 12.5 -> 5.51 mm, vias 2 -> 0
- net Net-(J5-Pin_15): track 6.75 -> 0.00 mm
- net /MCU_RF_RST: track 4.66 -> 0.00 mm
- net /RF_I2S_DFS: track 6.58 -> 2.01 mm
- net /MCU_I2S_SDIO: track 3.53 -> 0.00 mm
- net /MCU_RF_SEN: track 3.29 -> 0.00 mm
- net /RF_I2S_DCLK: track 5.42 -> 2.16 mm
- net Net-(U2-LO-): track 3.23 -> 0.00 mm
- net /RF_I2S_DOUT: track 5.88 -> 2.83 mm
- net Net-(U2-LO+): track 2.73 -> 0.00 mm
- net /MCU_I2C_SCLK: track 2.59 -> 0.00 mm
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- added copper zone on F.Cu, net GND
- removed copper zone on In1.Cu, net GND
