File: ECE362_4_Layer/ECE362_4_Layer.kicad_sch (KiCad schematic)
At the start: 54 parts, among them IC1 SI4705-D62-GM, J1 SPEAKER OUT, P1 USB_C_Plug_USB2.0, SW1 SW_Push, SW2 SW_Push, U1 W25Q128JVS, U3 LD1117S33TR_SOT223, U4 TL071, U5 PAM8302AAS, U6 RP2350B-QFN80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

Commit message: Changed RF input to headers
Parts:
- removed C24: 10pF, Capacitor_SMD:C_0201_0603Metric, symbol Device:C
- removed C25: 22nF, symbol Device:C
- removed C26: 1nF, symbol Device:C
- removed C27: 100nF, symbol Device:C
- removed IC1: SI4705-D62-GM, SI4705D62GM, symbol SI4705-D62-GM:SI4705-D62-GM
- removed R14, R15: 10k, symbol Device:R
- removed U5: PAM8302AAS, Package_SO:MSOP-8_3x3mm_P0.65mm, symbol Amplifier_Audio:PAM8302AAS
- added C30: 0.05, Capacitor_SMD:C_0201_0603Metric, symbol Device:C
- added C31: 250uF, Capacitor_SMD:C_0201_0603Metric, symbol Device:C
- added J3: Conn_01x02_Pin, symbol Connector:Conn_01x02_Pin
- added J4: Conn_01x08_Pin, symbol Connector:Conn_01x08_Pin
- added R16: 10, symbol Device:R
- added U7: LM386, symbol Amplifier_Audio:LM386
- C8: value 10uF -> .1uF
Connections:
- net +3.3V: now also J4.2 (Pin_2), U7.6 (V+)
- net GND: now also J1.2 (Pin_2), J4.1 (Pin_1), R16.2, U7.2 (-), U7.4 (GND)
- net at C11.2: now also U7.3 (+)
- net at J1.1 (Pin_1): now also C31.2
- net LOUT renamed RF_LIN
- net RF_LIN: now also J3.2 (Pin_2)
- net ROUT renamed RF_RIN
- net RF_RIN: now also J3.1 (Pin_1)
- new net: C30.1, C31.1, U7.5
- new net: C30.2, R16.1
- new net RF_GPIO_1: J4.7 (Pin_7)
- new net RF_GPIO_2: J4.8 (Pin_8)
- new net SCLK: J4.4 (Pin_4)
- new net SDIO: J4.3 (Pin_3)
- new net ~{RST}: J4.6 (Pin_6)
- new net ~{SEN}: J4.5 (Pin_5)
- no-connect marks 1 -> 0
Other:
- note removed: "Audio power amplifier. 4Ohm rated output impedance."
- moved on the sheet: C13, C14, J1
