File: RF_INPUT_BREAKOUT/RF_INPUT_BREAKOUT.kicad_sch (KiCad schematic)
At the start: 18 parts, among them IC1 SI4705-D62-GM, J1 5V Input, J2 I2C, J3 I2C, U1 LD1117S33TR_SOT223, U2 LT5512EUF-PBF, U3 Si5351A-B-GT

Commit message: Did added external osc
Parts:
- removed U3: Si5351A-B-GT, Package_SO:MSOP-10_3x3mm_P0.5mm, symbol Oscillator:Si5351A-B-GT
- added J4: RF IN, symbol Connector:Conn_Coaxial_Small
- added R4: 10k, symbol Device:R
- added X1: ASE-xxxMHz, Oscillator:Oscillator_SMD_Abracon_ASE-4Pin_3.2x2.5mm, symbol Oscillator:ASE-xxxMHz
- C7: value .47uF -> 1uF
- C8: value .47uF -> .01uF
- J3: value I2C -> MCU_RF_RCLK
- R1, R2: value 10k -> 4.7k
Connections:
- net +3.3V: now also R4.1; no longer C7.1, C8.1
- net +5V: now also C7.1, C8.1, U2.6 (VCC1), U2.7 (VCC2)
- net GND: now also IC1.3 (RFGND), U2.10 (IF-), U2.17 (EP), U2.3 (RF-), J4.2 (Ext)
- net IF_OUT: now reaches U2.11 (IF+)
- net at U2.2 (RF+): now also J4.1 (In)
- net DC_EN: now reaches U2.5 (EN)
- net LO_CLK: now reaches C5.1
- net RF_ANALOG_ROUT: now reaches IC1.13 (ROUT/[DOUT])
- net RF_ANALOG_LOUT: now reaches IC1.14 (LOUT/[DFS])
- net RF_I2S_DOUT: now reaches IC1.15 (DOUT)
- net RF_I2S_DFS: now reaches IC1.16 (DFS)
- net RF_I2S_DCLK: now reaches IC1.17 (GPO3/[DCLK])
- net MCU_RF_RST: now reaches IC1.5 (~{RST})
- net MCU_RF_SEN: now reaches IC1.6 (~{SEN})
- net MCU_RF_SEN: now also R4.2
- net RCLK renamed MCU_RF_RCLK
Other:
- moved on the sheet: C1, C2, C3, C4, C5, C6, IC1, J1, J2, J3, R1, R2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

Commit message: added headers
Parts:
- removed J2: I2C, symbol Connector:Conn_01x02_Pin
- removed J3: MCU_RF_RCLK, symbol Connector:Conn_01x02_Pin
- added C10, C11: 1uF, Capacitor_SMD:C_0402_1005Metric, symbol Device:C
- added C9: 33pF, Capacitor_SMD:C_0402_1005Metric, symbol Device:C
- added J5: Conn_2Rows-21Pins, Connector_PinHeader_1.00mm:PinHeader_2x11_P1.00mm_Vertical, symbol Connector_Generic:Conn_2Rows-21Pins
- added L1, L2: 12nH, Inductor_SMD:L_0402_1005Metric, symbol Device:L
- added R10, R7, R8, R9: 330, Resistor_SMD:R_0402_1005Metric, symbol Device:R
- added R5, R6: 10k, Resistor_SMD:R_0402_1005Metric, symbol Device:R
- added T1: Transformer_1P_SS, symbol Device:Transformer_1P_SS
- C1: footprint (none) -> Capacitor_SMD:C_1206_3216Metric
- C2, C7: footprint (none) -> Capacitor_SMD:C_0201_0603Metric
- C3, C4, C5, C6, C8: footprint (none) -> Capacitor_SMD:C_0402_1005Metric
- IC1: footprint SI4705D62GM -> Package_DFN_QFN:QFN-20-1EP_3x3mm_P0.4mm_EP1.65x1.65mm
- R1, R2, R3, R4: footprint (none) -> Resistor_SMD:R_0402_1005Metric
- U2: footprint QFN-16_UF_LIT -> Package_DFN_QFN:QFN-16-1EP_4x4mm_P0.5mm_EP2.45x2.45mm
Connections:
- net +5V: now also J5.1 (Pin_1)
- net GND: now also J5.10 (Pin_10), J5.12 (Pin_12), J5.14 (Pin_14), J5.16 (Pin_16), J5.18 (Pin_18), J5.20 (Pin_20), J5.3 (Pin_3), J5.4 (Pin_4), J5.6 (Pin_6), J5.8 (Pin_8), R5.2, R6.2, T1.2 (AB), T1.4 (SC); no longer U2.3 (RF-)
- net MCU_RF_RST: now also R10.1, R5.1
- net MCU_RF_SEN: now also R9.1
- net RF_ANALOG_LOUT: now also C11.1, J5.11 (Pin_11); no longer IC1.14 (LOUT/[DFS])
- net RF_ANALOG_ROUT: now also C10.1, J5.13 (Pin_13); no longer IC1.13 (ROUT/[DOUT])
- net RF_I2S_DCLK: now also J5.5 (Pin_5)
- net RF_I2S_DFS: now also J5.7 (Pin_7)
- net RF_I2S_DOUT: now also J5.9 (Pin_9)
- net at U2.2 (RF+): now also L1.2; no longer J4.1 (In)
- net MCU_I2C_SCLK: now reaches IC1.8 (SDIO), R2.2
- net MCU_I2C_SCLK: now also IC1.7 (SCLK), R1.2, R7.1, R8.1
- net DC_EN renamed MCU_MIX_EN 3V
- net MCU_MIX_EN 3V: now also J5.2 (Pin_2), R6.1
- new net: C11.2, IC1.14 (LOUT/[DFS])
- new net: L2.2, U2.3 (RF-)
- new net: J4.1 (In), T1.1 (AA)
- new net: C10.2, IC1.13 (ROUT/[DOUT])
- new net: C9.1, L1.1, T1.5 (SB)
- new net: J5.15 (Pin_15), R7.2
- new net: C9.2, L2.1, T1.3 (SA)
- new net: J5.19 (Pin_19), R9.2
- new net: J5.17 (Pin_17), R8.2
- new net: J5.21 (Pin_21), R10.2
Other:
- moved on the sheet: C1, C2, C3, C4, C5, C6, C7, C8, IC1, J1, J4, R1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

Commit message: redid layout
Parts:
- removed R1, R2: 4.7k, Resistor_SMD:R_0402_1005Metric, symbol Device:R
- added J2: Conn_01x02_Pin, symbol Connector:Conn_01x02_Pin
Connections:
- net +5V: now also J2.1 (Pin_1); no longer J5.1 (Pin_1)
- net GND: now also J5.1 (Pin_1), J2.2 (Pin_2); no longer J5.3 (Pin_3)
- net MCU_I2C_SCLK: no longer IC1.8 (SDIO), R7.1
- net MCU_RF_RCLK: now also J5.13 (Pin_13)
- net RF_ANALOG_LOUT: now also J5.9 (Pin_9); no longer J5.11 (Pin_11)
- net RF_ANALOG_ROUT: now also J5.11 (Pin_11); no longer J5.13 (Pin_13)
- net RF_I2S_DCLK: now also J5.3 (Pin_3); no longer J5.5 (Pin_5)
- net RF_I2S_DFS: now also J5.5 (Pin_5); no longer J5.7 (Pin_7)
- net RF_I2S_DOUT: now also J5.7 (Pin_7); no longer J5.9 (Pin_9)
- new net MCU_I2S_SDIO: IC1.8 (SDIO), R7.1
Other:
- moved on the sheet: J5, R10, R7, R8, R9

Commit message: switched for LT5560 Mixer
Parts:
- removed U2: LT5512EUF-PBF, Package_DFN_QFN:QFN-16-1EP_4x4mm_P0.5mm_EP2.45x2.45mm, symbol 2025-09-15_19-51-34:LT5512EUF-PBF
- removed X1: ASE-xxxMHz, Oscillator:Oscillator_SMD_Abracon_ASE-4Pin_3.2x2.5mm, symbol Oscillator:ASE-xxxMHz
- added L3: 180nH, Inductor_SMD:L_0402_1005Metric, symbol Device:L
- added T2: ADT16-1, symbol Device:Transformer_1P_SS
- added U2: LT5560, Package_DFN_QFN:DFN-8-1EP_3x3mm_P0.5mm_EP1.66x2.38mm, symbol RF_Mixer:LT5560
- C7: value 1uF -> 1nF; footprint Capacitor_SMD:C_0201_0603Metric -> Capacitor_SMD:C_0402_1005Metric
- C8: value .01uF -> 1uF; footprint Capacitor_SMD:C_0402_1005Metric -> Capacitor_SMD:C_0603_1608Metric
- C9: value 33pF -> 22pF
- IC1: footprint Package_DFN_QFN:QFN-20-1EP_3x3mm_P0.4mm_EP1.65x1.65mm -> Package_DFN_QFN:QFN-20-1EP_4x4mm_P0.5mm_EP2.5x2.5mm
- L1, L2: value 12nH -> 18nH
- T1: value Transformer_1P_SS -> WBC 1-1
Connections:
- net +3.3V: now also C7.1, C8.1, T2.4 (SC), U2.7 (VCC)
- net +5V: no longer C7.1, C8.1
- net GND: now also L3.1, T2.2 (AB), U2.9 (PGND)
- net IF_OUT: now also IC1.2 (FMI), L3.2, T2.1 (AA)
- net MCU_MIX_EN 3V: now also U2.2 (EN)
- net at L1.2: now also U2.3 (IN+)
- net at L2.2: now also U2.4 (IN-)
- new net: T2.3 (SA), U2.5 (OUT-)
- new net: T2.5 (SB), U2.6 (OUT+)
Other:
- moved on the sheet: C1, C10, C11, C2, C3, C4, C5, C6, C9, IC1, J1, J2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

Commit message: added PLL and VCO, need to finish Loop filter
Parts:
- removed J2: Conn_01x02_Pin, symbol Connector:Conn_01x02_Pin
- added C12, C16: 1nF, Capacitor_SMD:C_0603_1608Metric, symbol Device:C
- added C13: 10uF, Capacitor_SMD:C_0201_0603Metric, symbol Device:C
- added C14, C15: 12pF, Capacitor_SMD:C_0201_0603Metric, symbol Device:C
- added IC2: MAX2606EUT+T, SOT95P280X145-6N, symbol MAX2606EUT+T:MAX2606EUT+T
- added L4: 1.2uH, Inductor_SMD:L_0402_1005Metric, symbol Device:L
- added L6, L7: 680nH, Inductor_SMD:L_1008_2520Metric, symbol Device:L
- added R1: 10, Resistor_SMD:R_0603_1608Metric, symbol Device:R
- added R11: 10k, Resistor_SMD:R_0603_1608Metric, symbol Device:R
- added R12: 11k, Resistor_SMD:R_0603_1608Metric, symbol Device:R
- added R2: 270, Resistor_SMD:R_0603_1608Metric, symbol Device:R
- added U3: ADF4002BRUZ, Package_SO:TSSOP-16_4.4x5mm_P0.65mm, symbol Timer_PLL:ADF4002BRUZ
- C5, C6: value .01uF -> 10nF
- J4: footprint (none) -> Connector_Coaxial:SMA_Amphenol_132289_EdgeMount
- R3: value 100 -> 160
Connections:
- net +3.3V: now also C13.1, R1.2, R11.2
- net GND: now also C6.1, R3.2, C12.2, C13.2, C15.2, C16.2, IC2.2 (GND), IC2.4 (OUT-), L4.1, L7.1; no longer C6.2
- net MCU_I2C_SCLK: now also U3.11 (CLK)
- net MCU_I2S_SDIO: now also U3.12 (DATA)
- net at C5.2, R3.1: now also U2.1 (LO-)
- net at U2.8 (LO+): now also C6.2
- net LO_CLK renamed RF_MIX_LO
- new net: IC2.1 (IND), L4.2
- new net: C12.1, IC2.3 (TUNE), R2.2
- new net: C16.1, IC2.5 (VCC), L6.1, L7.2, R1.1
- new net: C14.2, IC2.6 (OUT+), L6.2
- new net: R11.1, R12.2
- new net VCO_PLL_RFINA: C14.1, U3.6 (RFINA)
- new net VCO_PLL_RFINB: C15.1, U3.5 (RFINB)
- new net VCO_TUNE: R2.1
Other:
- note added: "MAIN BOARD CONNECTION"
- note added: "MIN Q = 35"
- note added: "NPO/C0G Cap ONLY"
- note added: "POWER SUPPLY"
- note added: "RF MIXER LT5560"
- note added: "RF TUNER Si4705"
- company: (none) -> ECE_36200
- title: (none) -> SSTV RF BREAKOUT BOARD
- moved on the sheet: C1, C10, C11, C2, C3, C4, C5, C7, C8, C9, IC1, J1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

Commit message: slight changes
Parts:
- removed L7: 680nH, Inductor_SMD:L_1008_2520Metric, symbol Device:L
- added C17, C18, C19, C20: 100pF, Capacitor_SMD:C_0603_1608Metric, symbol Device:C
- added R13, R14: 4.7k, Resistor_SMD:R_0402_1005Metric, symbol Device:R
- added R15: 1k, Resistor_SMD:R_0402_1005Metric, symbol Device:R
- added R16: 50, Resistor_SMD:R_0603_1608Metric, symbol Device:R
- R11: footprint Resistor_SMD:R_0603_1608Metric -> Resistor_SMD:R_0402_1005Metric
- R12: value 11k -> 10k; footprint Resistor_SMD:R_0603_1608Metric -> Resistor_SMD:R_0402_1005Metric
Connections:
- net +3.3V: now also U3.16 (VP), C20.1, R13.2, R14.2, R15.1; no longer R11.2
- net GND: now also R11.2, R12.2, U3.3 (CPGND), U3.4 (AGND), U3.9 (DGND), C17.2, C18.2, C19.2, C20.2; no longer C15.2, IC2.4 (OUT-)
- net VCO_PLL_RFINA: now also C15.1; no longer C14.1
- net at C16.1, IC2.5 (VCC), L6.1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: now also R16.2
- net at U3.1 (RSET): now also R11.1
- net at U3.15 (DVDD): now also R12.1, U3.7 (AVDD), C18.1, C19.1, R15.2
- net at J5.15 (Pin_15), R7.2: now also R13.1
- net at J5.17 (Pin_17), R8.2: now also R14.1
- net RF_MIX_LO renamed VCO_MIXER_OUT
- net VCO_MIXER_OUT: now also C14.1
- net VCO_PLL_RFINB: no longer names the net of U3.5 (RFINB)
- net VCO_PLL_RFINB: now also C17.1; no longer C15.1
- new net: C15.2, IC2.4 (OUT-), R16.1
Other:
- moved on the sheet: C12, C13, C14, C15, C16, IC2, L4, L6, R1, R2, R7, R8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

Commit message: meeting 9/21
Parts:
- added C21, C22: .1uF, Capacitor_SMD:C_0603_1608Metric, symbol Device:C
- added Y1: ASE-60MHz, Oscillator:Oscillator_SMD_Abracon_ASE-4Pin_3.2x2.5mm, symbol Oscillator:ASE-xxxMHz
- C15: value 12pF -> 1nF
- C19: value 100pF -> .1uF
Connections:
- net +3.3V: now also C21.1, Y1.1 (EN), Y1.4 (Vdd)
- net GND: now also C21.2, Y1.2 (GND)
- net at U3.8 (REFIN): now also C22.1
- new net: C22.2, Y1.3 (OUT)
Other:
- moved on the sheet: C1, C12, C13, C14, C15, C16, C17, C18, C19, C2, C20, IC2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

Commit message: some stuff
Connections:
- net MCU_I2S_SDIO: no longer U3.12 (DATA)
- new net MCU_I2C_SDIO: U3.12 (DATA)
Other:
- moved on the sheet: C12, C13, C14, C15, C16, IC2, L4, L6, R1, R16, R2
