File: RF_INPUT_BREAKOUT_SIMPLE/RF_INPUT_BREAKOUT_SIMPLE.kicad_pcb (KiCad board)
At the start: 2 copper layers, 97.5 x 108.2 mm, 27 parts, among them J1 KEYPAD, J10 ROTARY ENCODER, J2 Conn_01x28_Pin, J3 DebugnBoot, J4 Conn_01x28_Pin, J5 OLED, J6 AUDIO_JACK, J7 UART-PINS, J8 OLED SPI, J9 SI4703

Commit message: Layout Adjustments
Parts:
- moved R14 46.0 mm to (135.5, 107.6)
- moved J10 40.2 mm to (190.5, 57.0)
- moved J5 15.5 mm to (103.0, 118.7)
- moved C2 15.5 mm to (110.2, 153.1)
- moved C3 15.5 mm to (107.2, 153.1)
- moved J8 15.5 mm to (187.2, 131.4)
- moved J9 3.68 mm to (146.8, 77.0)
Routing:
- net +3V3: track 224.5 -> 264.1 mm, vias 1 -> 0
- net /ROT_SW: track 48.8 -> 67.6 mm
- net /ROT_DT: track 48.8 -> 67.6 mm
- net /ROT_CLK: track 48.8 -> 67.6 mm
- net /OLED_SPI0_~{RST}: track 39.6 -> 56.4 mm
- net /OLED_SPI0_CS: track 36.8 -> 49.0 mm
- net /OLED_SPI1_RX: track 50.3 -> 62.3 mm
- net /OLED_SPI0_TX: track 23.4 -> 34.4 mm
- net /OLED_SPI0_SCK: track 23.4 -> 34.4 mm
- net /OLED_DC: track 23.4 -> 34.4 mm
- net /OLED_SPI1_TX: track 50.3 -> 56.7 mm
- net /OLED_SPI1_SCLK: track 51.3 -> 57.7 mm
- net /OLED_SPI1_CS: track 58.5 -> 64.9 mm
- net /RF_SDIO: track 12.0 -> 8.24 mm
- net /RF_SCLK: track 12.0 -> 8.24 mm
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
Commit message: changed SMD components to 0805
Parts:
- C1, C2, C3: footprint Capacitor_SMD:C_0603_1608Metric -> Capacitor_SMD:C_0805_2012Metric
- R1, R10, R11, R12, R13, R14, R2, R3, R4, R5, R6, R7, R8, R9: footprint Resistor_SMD:R_0603_1608Metric -> Resistor_SMD:R_0805_2012Metric
- moved R9 0.70 mm to (115.8, 73.8)
- moved C2 0.33 mm to (110.2, 152.8)
- moved C3 0.33 mm to (107.2, 152.8)
- moved R7 0.09 mm to (108.3, 81.2)
Routing:
- net GND: vias 66 -> 114
