File: RF_INPUT_BREAKOUT_SIMPLE/RF_INPUT_BREAKOUT_SIMPLE.kicad_sch (KiCad schematic)
At the start: 1 part, among them J1 Si4703 Breakout Board

Commit message: some stuff
Parts:
- removed J1: Si4703 Breakout Board, Connector_Hirose:Hirose_DF13-10P-1.25DSA_1x10_P1.25mm_Vertical, symbol Connector:Conn_01x10_Pin
- added J2, J4: Conn_01x28_Pin, Connector_PinHeader_2.54mm:PinHeader_1x28_P2.54mm_Vertical, symbol Connector:Conn_01x28_Pin
- added J3: DebugnBoot, Connector_PinHeader_2.54mm:PinHeader_1x04_P2.54mm_Vertical, symbol Connector:Conn_01x04_Pin
- added J5: Si4703, symbol Connector:Conn_01x08_Socket
- added J7: UART-PINS, Connector_PinHeader_2.54mm:PinHeader_1x03_P2.54mm_Vertical, symbol Connector:Conn_01x03_Pin
Connections:
- net GND: now also J2.28 (Pin_28), J4.28 (Pin_28), J5.7 (Pin_7)
- net GPIO1: now also J2.4 (Pin_4), J7.1 (Pin_1)
- net GPIO2: now also J2.5 (Pin_5)
- new net +3V3: J2.2 (Pin_2), J4.2 (Pin_2), J5.8 (Pin_8)
- new net GPIO0: J2.3 (Pin_3), J7.3 (Pin_3)
- new net GPIO10: J2.13 (Pin_13)
- new net GPIO11: J2.14 (Pin_14)
- new net GPIO12: J2.15 (Pin_15)
- new net GPIO13: J2.16 (Pin_16)
- new net GPIO14: J2.17 (Pin_17)
- new net GPIO15: J2.18 (Pin_18)
- new net GPIO16: J2.19 (Pin_19)
- new net GPIO17: J2.20 (Pin_20)
- new net GPIO18: J2.21 (Pin_21)
- new net GPIO19: J2.22 (Pin_22)
- new net GPIO20: J2.23 (Pin_23)
- new net GPIO21: J2.24 (Pin_24)
- new net GPIO22: J2.25 (Pin_25)
- new net GPIO23: J2.26 (Pin_26)
- new net GPIO24: J2.27 (Pin_27)
- new net GPIO25: J4.25 (Pin_25)
- new net GPIO26: J4.24 (Pin_24)
- new net GPIO27: J4.23 (Pin_23)
- new net GPIO28: J4.22 (Pin_22)
- new net GPIO29: J4.21 (Pin_21)
- new net GPIO3: J2.6 (Pin_6)
- new net GPIO30: J4.20 (Pin_20)
- new net GPIO31: J4.19 (Pin_19)
- new net GPIO32: J4.18 (Pin_18)
- new net GPIO33: J4.17 (Pin_17)
- new net GPIO34: J4.16 (Pin_16)
- new net GPIO35: J4.15 (Pin_15)
- new net GPIO36: J4.14 (Pin_14)
- new net GPIO37: J4.13 (Pin_13)
- new net GPIO38: J4.12 (Pin_12)
- new net GPIO39: J4.11 (Pin_11)
- new net GPIO4: J2.7 (Pin_7)
- new net GPIO40_ADC0: J4.10 (Pin_10)
- new net GPIO41_ADC1: J4.9 (Pin_9)
- new net GPIO42_ADC2: J4.8 (Pin_8)
- new net GPIO43_ADC3: J4.7 (Pin_7)
- new net GPIO44_ADC4: J4.6 (Pin_6)
- new net GPIO45_ADC5: J4.5 (Pin_5)
- new net GPIO46_ADC6: J4.4 (Pin_4)
- new net GPIO47_ADC7: J4.3 (Pin_3)
- new net GPIO5: J2.8 (Pin_8)
- new net GPIO6: J2.9 (Pin_9)
- new net GPIO7: J2.10 (Pin_10)
- new net GPIO8: J2.11 (Pin_11)
- new net GPIO9: J2.12 (Pin_12)
- new net RF_GPIO1: J5.2 (Pin_2)
- new net RF_GPIO2: J5.1 (Pin_1)
- new net RF_SCLK: J5.4 (Pin_4)
- new net RF_SDIO: J5.3 (Pin_3)
- new net RF_SEN: J5.5 (Pin_5)
- new net RF_~{RST}: J5.6 (Pin_6)
- new net SWCLK: J4.26 (Pin_26)
- new net SWD: J4.27 (Pin_27)
- new net VBUS: J2.1 (Pin_1), J4.1 (Pin_1)

Commit message: adding breakouts
Parts:
- added C1: 47nF, symbol Device:C
- added J1: KEYPAD, symbol Connector:Conn_01x08_Socket
- added J6: AUDIO_JACK, Connector_PinHeader_2.54mm:PinHeader_1x04_P2.54mm_Vertical, symbol Connector:Conn_01x04_Pin
- added J8: ROTARY ENCODER, symbol Connector:Conn_01x05_Socket
- added R1, R13, R2, R3, R4, R5, R6, R7, R8: 1k, symbol Device:R
- added R10, R11, R12, R9: 10k, symbol Device:R
Connections:
- net GPIO36 is gone; now on net RF_SDIO: J4.14 (Pin_14)
- net GPIO37 is gone; now on net RF_SCLK: J4.13 (Pin_13)
- net GPIO40_ADC0 is gone; now on net RF_~{RST}: J4.10 (Pin_10)
- net GND: now also J7.2 (Pin_2), C1.2, J6.1 (Pin_1), R10.1, R11.1, R12.1, R9.1
- net GPIO2: now also R1.2, R12.2
- net GPIO3: now also R11.2, R2.2
- net GPIO4: now also R10.2, R3.2
- net GPIO41_ADC1: now also C1.1, R13.1
- net GPIO5: now also R4.2, R9.2
- net GPIO6: now also R5.2
- net GPIO7: now also R6.2
- net GPIO8: now also R7.2
- net GPIO9: now also R8.2
- net RF_SCLK: now also J5.5 (Pin_5); no longer J5.4 (Pin_4)
- net RF_SDIO: now also J5.6 (Pin_6); no longer J5.3 (Pin_3)
- net RF_SEN: now also J5.4 (Pin_4); no longer J5.5 (Pin_5)
- net RF_~{RST}: now also J5.3 (Pin_3); no longer J5.6 (Pin_6)
- new net: J1.8 (Pin_8), R8.1
- new net: J6.4 (Pin_4), R13.2
- new net: J1.3 (Pin_3), R3.1
- new net: J1.4 (Pin_4), R4.1
- new net: J1.7 (Pin_7), R7.1
- new net: J1.6 (Pin_6), R6.1
- new net: J1.5 (Pin_5), R5.1
- new net: J1.1 (Pin_1), R1.1
- new net: J1.2 (Pin_2), R2.1
- new net CLK: J8.1 (Pin_1)
- new net DT: J8.2 (Pin_2)
- new net SW: J8.3 (Pin_3)
Other:
- moved on the sheet: J2, J3, J4, J5, J7

Commit message: Finished Layout
Parts:
- removed J1: KEYPAD, symbol Connector:Conn_01x08_Socket
- removed J5: Si4703, symbol Connector:Conn_01x08_Socket
- removed J8: ROTARY ENCODER, symbol Connector:Conn_01x05_Socket
- added C2: 10uF, Capacitor_SMD:C_0603_1608Metric, symbol Device:C
- added C3: .1uF, Capacitor_SMD:C_0603_1608Metric, symbol Device:C
- added J1: KEYPAD, Connector_PinHeader_2.54mm:PinHeader_1x08_P2.54mm_Vertical, symbol Connector:Conn_01x08_Pin
- added J10: ROTARY ENCODER, Connector_PinHeader_2.54mm:PinHeader_1x05_P2.54mm_Vertical, symbol Connector:Conn_01x05_Pin
- added J5: OLED, Connector_PinHeader_2.54mm:PinHeader_1x14_P2.54mm_Vertical, symbol Connector:Conn_01x14_Pin
- added J8: OLED SPI, Connector_PinHeader_2.54mm:PinHeader_1x04_P2.54mm_Vertical, symbol Connector:Conn_01x04_Pin
- added J9: SI4703, Connector_PinHeader_2.54mm:PinHeader_1x08_P2.54mm_Vertical, symbol Connector:Conn_01x08_Pin
- added R14: 10k, Resistor_SMD:R_0603_1608Metric, symbol Device:R
- C1: footprint (none) -> Capacitor_SMD:C_0603_1608Metric
- R1, R10, R11, R12, R13, R2, R3, R4, R5, R6, R7, R8, R9: footprint (none) -> Resistor_SMD:R_0603_1608Metric
Connections:
- net +3V3: now also C2.1, C3.1, J10.4 (Pin_4), J5.14 (Pin_14), J5.7 (Pin_7), J9.8 (Pin_8), R14.2
- net GND: now also C2.2, C3.2, J10.5 (Pin_5), J5.13 (Pin_13), J9.7 (Pin_7)
- net RF_GPIO1: now also J9.2 (Pin_2)
- net RF_GPIO2: now also J9.1 (Pin_1)
- net RF_SCLK: now also J9.5 (Pin_5)
- net RF_SDIO: now also J9.6 (Pin_6)
- net RF_SEN: now also J9.4 (Pin_4)
- net RF_~{RST}: now also J9.3 (Pin_3)
- net at R8.1: now also J1.8 (Pin_8)
- net at R3.1: now also J1.3 (Pin_3)
- net at R4.1: now also J1.4 (Pin_4)
- net at R7.1: now also J1.7 (Pin_7)
- net at R6.1: now also J1.6 (Pin_6)
- net at R5.1: now also J1.5 (Pin_5)
- net at R1.1: now also J1.1 (Pin_1)
- net at R2.1: now also J1.2 (Pin_2)
- net GPIO16 renamed OLED_SPI0_~{RST}
- net OLED_SPI0_~{RST}: now also J5.11 (Pin_11)
- net GPIO17 renamed OLED_SPI0_CS
- net OLED_SPI0_CS: now also J5.12 (Pin_12)
- net GPIO18 renamed OLED_SPI0_SCK
- net OLED_SPI0_SCK: now also J5.8 (Pin_8)
- net GPIO19 renamed OLED_SPI0_TX
- net OLED_SPI0_TX: now also J5.9 (Pin_9)
- net GPIO20 renamed OLED_DC
- net OLED_DC: now also J5.10 (Pin_10)
- net GPIO27 renamed OLED_SPI1_TX
- net OLED_SPI1_TX: now also J8.3 (Pin_3)
- net GPIO28 renamed OLED_SPI1_RX
- net OLED_SPI1_RX: now also J8.2 (Pin_2), R14.1
- net GPIO29 renamed OLED_SPI1_CS
- net OLED_SPI1_CS: now also J8.4 (Pin_4)
- net GPIO30 renamed OLED_SPI1_SCLK
- net OLED_SPI1_SCLK: now also J8.1 (Pin_1)
- net GPIO32 renamed ROT_SW
- net ROT_SW: now also J10.3 (Pin_3)
- net GPIO33 renamed ROT_DT
- net ROT_DT: now also J10.2 (Pin_2)
- net GPIO34 renamed ROT_CLK
- net ROT_CLK: now also J10.1 (Pin_1)
Other:
- moved on the sheet: C1, J3, J6, R13

Commit message: changed SMD components to 0805
Parts:
- C1, C2, C3: footprint Capacitor_SMD:C_0603_1608Metric -> Capacitor_SMD:C_0805_2012Metric
- R1, R10, R11, R12, R13, R14, R2, R3, R4, R5, R6, R7, R8, R9: footprint Resistor_SMD:R_0603_1608Metric -> Resistor_SMD:R_0805_2012Metric
Changed lines of the file:
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@@
 			)
 		)
-		(property "Footprint" "Resistor_SMD:R_0603_1608Metric"
+		(property "Footprint" "Resistor_SMD:R_0805_2012Metric"
 			(at 40.64 53.848 90)
 			(effects
@@
 			)
 		)
-		(property "Footprint" "Resistor_SMD:R_0603_1608Metric"
+		(property "Footprint" "Resistor_SMD:R_0805_2012Metric"
 			(at 83.058 57.15 90)
 			(effects
@@
 			)
 		)
-		(property "Footprint" "Capacitor_SMD:C_0603_1608Metric"
+		(property "Footprint" "Capacitor_SMD:C_0805_2012Metric"
 			(at 41.6052 151.13 0)
 			(effects
@@
 			)
 		)
-		(property "Footprint" "Resistor_SMD:R_0603_1608Metric"
+		(property "Footprint" "Resistor_SMD:R_0805_2012Metric"
 			(at 66.04 41.148 90)
 			(effects
@@
 			)
 		)
-		(property "Footprint" "Resistor_SMD:R_0603_1608Metric"
+		(property "Footprint" "Resistor_SMD:R_0805_2012Metric"
 			(at 75.438 69.85 90)
 			(effects
@@
 			)
 		)
-		(property "Footprint" "Resistor_SMD:R_0603_1608Metric"
+		(property "Footprint" "Resistor_SMD:R_0805_2012Metric"
 			(at 60.96 43.688 90)
 			(effects
@@
 			)
 		)
-		(property "Footprint" "Resistor_SMD:R_0603_1608Metric"
+		(property "Footprint" "Resistor_SMD:R_0805_2012Metric"
 			(at 71.628 76.2 90)
 			(effects
@@
 			)
 		)
-		(property "Footprint" "Capacitor_SMD:C_0603_1608Metric"
+		(property "Footprint" "Capacitor_SMD:C_0805_2012Metric"
 			(at 53.0352 151.13 0)
 			(effects
@@
 			)
 		)
-		(property "Footprint" "Resistor_SMD:R_0603_1608Metric"
+		(property "Footprint" "Resistor_SMD:R_0805_2012Metric"
 			(at 45.72 51.308 90)
 			(effects
@@
 			)
 		)
-		(property "Footprint" "Resistor_SMD:R_0603_1608Metric"
+		(property "Footprint" "Resistor_SMD:R_0805_2012Metric"
 			(at 99.568 121.92 90)
 			(effects
@@
 			)
 		)
-		(property "Footprint" "Resistor_SMD:R_0603_1608Metric"
+		(property "Footprint" "Resistor_SMD:R_0805_2012Metric"
 			(at 79.248 63.5 90)
 			(effects
@@
 			)
 		)
-		(property "Footprint" "Resistor_SMD:R_0603_1608Metric"
+		(property "Footprint" "Resistor_SMD:R_0805_2012Metric"
 			(at 50.8 48.768 90)
 			(effects
@@
 			)
 		)
-		(property "Footprint" "Capacitor_SMD:C_0603_1608Metric"
+		(property "Footprint" "Capacitor_SMD:C_0805_2012Metric"
 			(at 214.3252 71.12 0)
 			(effects
@@
 			)
 		)
-		(property "Footprint" "Resistor_SMD:R_0603_1608Metric"
+		(property "Footprint" "Resistor_SMD:R_0805_2012Metric"
 			(at 220.98 64.008 90)
 			(effects
@@
 			)
 		)
-		(property "Footprint" "Resistor_SMD:R_0603_1608Metric"
+		(property "Footprint" "Resistor_SMD:R_0805_2012Metric"
 			(at 55.88 46.228 90)
 			(effects
@@
 			)
 		)
-		(property "Footprint" "Resistor_SMD:R_0603_1608Metric"
+		(property "Footprint" "Resistor_SMD:R_0805_2012Metric"
 			(at 71.12 38.608 90)
 			(effects
@@
 			)
 		)
-		(property "Footprint" "Resistor_SMD:R_0603_1608Metric"
+		(property "Footprint" "Resistor_SMD:R_0805_2012Metric"
 			(at 76.2 36.068 90)
 			(effects
