File: Proton-KiCAD/DebugProbe.kicad_sch (KiCad schematic)
At the start: 52 parts, among them J3 DebugnBoot, U10 USBLC6-2P6

Commit message: working on 4layer proton
Parts:
- removed J?: UART-PINS, Connector_PinHeader_2.54mm:PinHeader_1x03_P2.54mm_Vertical, symbol Connector:Conn_01x03_Pin
- gave numbers to parts that had none: 49
Connections:
- net UART_TX: now reaches R24.2
- net UART_RX: now reaches R25.2, R26.2

Commit message: did some layout
Parts:
- U5: renamed from U4; footprint W25Q16JVUXIQ:USON-8_UX_2x3x0p6_WIN -> Package_SON:Winbond_USON-8-1EP_3x2mm_P0.5mm_EP0.2x1.6mm
- U8: renamed from U6; footprint DebugProbe:RP2040-QFN-56 -> Package_DFN_QFN:QFN-56-1EP_7x7mm_P0.4mm_EP3.2x3.2mm
- U9: renamed from U7; footprint SN74AUP1T17DCKR:DCK5 -> Package_TO_SOT_SMD:Texas_R-PDSO-G5_DCK-5
- renumbered C24 to C22, C25 to C23, C26 to C24, C27 to C25, C29 to C26, C28 to C27, C30 to C28, C31 to C29, C32 to C30, C33 to C31, C34 to C32, C35 to C33, C36 to C34, C37 to C35, C38 to C36, C39 to C37, C40 to C38, C41 to C39, C42 to C40, J5 to J3, J3 to J4, R17 to R11, R23 to R12, R18 to R13, R19 to R14, R20 to R15, R21 to R16, R22 to R17, R24 to R18, R25 to R19, R26 to R20, R27 to R21, R28 to R22, R29 to R23, R30 to R24, R31 to R25, R32 to R26, R33 to R27, U8 to U10, U10 to U6, U5 to U7
