File: Proton-KiCAD/untitled.kicad_sch (KiCad schematic)
At the start: 16 parts, among them J10 ROTARY ENCODER, J2 AUDIO_JACK, J4 KEYPAD, J9 SI4703

Commit message: did some layout
Parts:
- removed J2: AUDIO_JACK, Connector_PinHeader_2.54mm:PinHeader_1x04_P2.54mm_Vertical, symbol Connector:Conn_01x04_Pin
- added C41: 0.1uF, Capacitor_SMD:C_0402_1005Metric, symbol Device:C
- added C42, C43: 22nF, Capacitor_SMD:C_0402_1005Metric, symbol Device:C
- added C44: 1uF, Capacitor_SMD:C_0402_1005Metric, symbol Device:C
- added C45: 0.05, Capacitor_SMD:C_0402_1005Metric, symbol Device:C
- added C46: 250uF, Capacitor_THT:CP_Radial_D10.0mm_P5.00mm, symbol Device:C
- added C47: 10uF, Capacitor_SMD:C_0805_2012Metric, symbol Device:C
- added C48: .1uF, Capacitor_SMD:C_0402_1005Metric, symbol Device:C
- added J10: OLED, Connector_PinHeader_2.54mm:PinHeader_1x14_P2.54mm_Vertical, symbol Connector:Conn_01x14_Pin
- added J6: RF_OUTPUT, Connector_Audio:Jack_3.5mm_CUI_SJ1-3525N_Horizontal, symbol Connector_Audio:AudioJack3_SwitchTR
- added J7: SPEAKER_OUT, Connector_PinHeader_2.54mm:PinHeader_1x02_P2.54mm_Vertical, symbol Connector:Conn_01x02_Pin
- added J8: OLED SPI, Connector_PinHeader_2.54mm:PinHeader_1x04_P2.54mm_Vertical, symbol Connector:Conn_01x04_Pin
- added R32, R40, R45, R47: 1k, Resistor_SMD:R_0402_1005Metric, symbol Device:R
- added R34, R48, R49: 100k, Resistor_SMD:R_0402_1005Metric, symbol Device:R
- added R35: 50k, Resistor_SMD:R_0402_1005Metric, symbol Device:R
- added R44, R46: 4k, Resistor_SMD:R_0402_1005Metric, symbol Device:R
- added R50: 10, Resistor_SMD:R_0402_1005Metric, symbol Device:R
- added R51: 10k, Resistor_SMD:R_0402_1005Metric, symbol Device:R
- added U11: TL072, Package_DIP:DIP-8_W7.62mm, symbol Amplifier_Operational:TL072
- added U12: LM386, Package_DIP:DIP-8_W7.62mm, symbol Amplifier_Audio:LM386
- R28, R42: renamed from R11; footprint Resistor_SMD:R_0805_2012Metric -> Resistor_SMD:R_0402_1005Metric
- R29, R43: renamed from R12; footprint Resistor_SMD:R_0805_2012Metric -> Resistor_SMD:R_0402_1005Metric
- R30: renamed from R13; footprint Resistor_SMD:R_0805_2012Metric -> Resistor_SMD:R_0402_1005Metric
- R31: renamed from R14; footprint Resistor_SMD:R_0805_2012Metric -> Resistor_SMD:R_0402_1005Metric
- R33: renamed from R15; footprint Resistor_SMD:R_0805_2012Metric -> Resistor_SMD:R_0402_1005Metric
- R36: renamed from R16; footprint Resistor_SMD:R_0805_2012Metric -> Resistor_SMD:R_0402_1005Metric
- R37: renamed from R34; footprint Resistor_SMD:R_0805_2012Metric -> Resistor_SMD:R_0402_1005Metric
- R38: renamed from R35; footprint Resistor_SMD:R_0805_2012Metric -> Resistor_SMD:R_0402_1005Metric
- R39: renamed from R36; footprint Resistor_SMD:R_0805_2012Metric -> Resistor_SMD:R_0402_1005Metric
- R41: renamed from R37; footprint Resistor_SMD:R_0805_2012Metric -> Resistor_SMD:R_0402_1005Metric
- renumbered J9 to J11, J4 to J5, J10 to J9
Connections:
- net +3V3: now also J9.4 (Pin_4), C47.1, C48.1, J10.14 (Pin_14), J10.7 (Pin_7), R51.2, U11.8 (V+)
- net GND: now also J9.5 (Pin_5), C42.2, C45.1, C47.2, C48.2, J10.13 (Pin_13), J6.S, J7.2 (Pin_2), R35.2, R45.2, R47.2, R49.2, U11.4 (V-), U12.2 (-), U12.4 (GND)
- new net: C46.1, J7.1 (Pin_1)
- new net: C46.2, R50.1, U12.5
- new net: C44.1, R46.2, R47.1
- new net: C44.2, R48.2, R49.1, U12.3 (+)
- new net: C41.1, J6.TN
- new net: C43.1, R34.1
- new net: C45.2, R50.2
- new net: C41.2, R32.1
- new net: R32.2, R40.1
- new net: R44.2, R45.1, U11.2 (-)
- new net: C42.1, R40.2, U11.3 (+)
- new net: R34.2, R35.1
- new net +5V: R48.1, U12.6 (V+)
- new net OLED_DC: J10.10 (Pin_10)
- new net OLED_SPI0_CS: J10.12 (Pin_12)
- new net OLED_SPI0_SCLK: J10.8 (Pin_8)
- new net OLED_SPI0_TX: J10.9 (Pin_9)
- new net OLED_SPI0_~{RST}: J10.11 (Pin_11)
- new net OLED_SPI1_CS: J8.4 (Pin_4)
- new net OLED_SPI1_RX: J8.2 (Pin_2), R51.1
- new net OLED_SPI1_SCLK: J8.1 (Pin_1)
- new net OLED_SPI1_TX: J8.3 (Pin_3)
- new net RF_AUDIO: C43.2, R44.1, R46.1, U11.1
Other:
- moved on the sheet: J11, J5, J9, R28, R29, R30, R31, R33, R36, R37, R38, R39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
