File: Proton-KiCAD/untitled.kicad_sch (KiCad schematic)
At the start: 42 parts, among them J10 OLED, J11 SI4703, J5 KEYPAD, J6 RF_OUTPUT, J7 SPEAKER_OUT, J8 OLED SPI, J9 ROTARY ENCODER, U11 TL072, U12 LM386

Commit message: Removing debugger
Parts:
- removed C24: 1uF, Capacitor_SMD:C_0402_1005Metric, symbol Device:C
- removed C41: 0.1uF, Capacitor_SMD:C_0402_1005Metric, symbol Device:C
- removed R34, R35, R48, R49: 100k, Resistor_SMD:R_0402_1005Metric, symbol Device:R
- removed R44: 10k, Resistor_SMD:R_0402_1005Metric, symbol Device:R
- removed R45: 90k, Resistor_SMD:R_0402_1005Metric, symbol Device:R
- added C22, C23, C27, C28: 47uF, Capacitor_SMD:C_0805_2012Metric, symbol Device:C
- added C30: 0.1uF, Capacitor_SMD:C_0402_1005Metric, symbol Device:C
- added R28, R29: 100k, Resistor_SMD:R_0402_1005Metric, symbol Device:R
- renumbered C42 to C24, C43 to C25, C44 to C26, C45 to C29, C46 to C31, C47 to C32, C48 to C33, J5 to J2, J6 to J3, J7 to J4, J8 to J5, J9 to J6, J10 to J7, J11 to J8, R28 to R11, R29 to R12, R30 to R13, R31 to R14, R32 to R15, R33 to R16, R36 to R17, R37 to R18, R38 to R19, R39 to R20, R40 to R21, R41 to R22, R42 to R23, R43 to R24, R52 to R25, R53 to R26, R50 to R27, R51 to R30, U11 to U5, U12 to U6
Connections:
- net +3V3: now also C22.1, R28.1
- net +5V: now also C27.1
- net GND: now also C22.2, C23.1, C27.2, C28.2, R29.2; no longer U5.4 (V-), U6.4 (GND)
- net RF_AUDIO: now also C30.2, R28.2, R29.1; no longer R25.1, U5.7
- net at C25.2, C26.1, U5.1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: now also U5.5 (+)
- net at J3.TN: now also R15.1
- new net: C23.2, U5.4 (V-)
- new net: C30.1, R25.1, U5.7
- new net: C28.1, U6.4 (GND)
Other:
- moved on the sheet: J3, R15, R25, R26, U5B, U5C

Commit message: need to spec audio jack
Parts:
- removed J3: RF_OUTPUT, Connector_Audio:Jack_3.5mm_CUI_SJ1-3525N_Horizontal, symbol Connector_Audio:AudioJack3_SwitchTR
- added J3: AudioJack3, Connector_Audio:Jack_3.5mm_CUI_SJ-3523-SMT_Horizontal, symbol Connector_Audio:AudioJack3
Connections:
- net GND: now also J3.S
- net at R15.1: now also J3.T
Other:
- moved on the sheet: C22, C23, C24, C25, C26, C27, C28, C29, C30, C31, J4, R15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

Commit message: ready for final check
Parts:
- added J11: FRONT_BUTTON_1, Connector_PinHeader_2.54mm:PinHeader_1x02_P2.54mm_Vertical, symbol Connector:Conn_01x02_Pin
- added J12: FRONT_BUTTON_2, Connector_PinHeader_2.54mm:PinHeader_1x02_P2.54mm_Vertical, symbol Connector:Conn_01x02_Pin
- added R31, R32: 1k, Resistor_SMD:R_0402_1005Metric, symbol Device:R
Connections:
- net GND: now also J11.2 (Pin_2), J12.2 (Pin_2)
- new net: J12.1 (Pin_1), R31.2
- new net: J11.1 (Pin_1), R32.2
- new net FRONT_BUTTON_1: R32.1
- new net FRONT_BUTTON_2: R31.1
Other:
- moved on the sheet: C32, C33, J5, J6, J7, R30

Commit message: Finished
Parts:
- removed J3: AudioJack3, Connector_Audio:Jack_3.5mm_CUI_SJ-3523-SMT_Horizontal, symbol Connector_Audio:AudioJack3
- added J3: SJ-43514, Custom_footprints:CUI_SJ-43514, symbol SJ-43514:SJ-43514
- C29: value 0.05 -> 0.05uF
- C31: value 250uF -> 200uF; footprint Capacitor_THT:CP_Radial_D10.0mm_P5.00mm -> Capacitor_SMD:CP_Elec_6.3x4.5
Connections:
- net GND: now also R27.2, J3.1; no longer C29.1
- net at C31.2, U6.5: now also C29.2; no longer R27.1
- net at R15.1: now also J3.2
- new net: C29.1, R27.1
Other:
- moved on the sheet: C29, C30, C31, J11, J12, J4, R27, R28, R29, R31

Commit message: fixed audio section
Parts:
- removed C28: 47uF, Capacitor_SMD:C_0805_2012Metric, symbol Device:C
- added R33: 1k, Resistor_SMD:R_0402_1005Metric, symbol Device:R
- added R34: 100k, Resistor_SMD:R_0402_1005Metric, symbol Device:R
- C27: value 47uF -> 0.1uF; footprint Capacitor_SMD:C_0805_2012Metric -> Capacitor_SMD:C_0402_1005Metric
Connections:
- net +5V: no longer C27.1
- net GND: now also C23.2, U5.4 (V-), U6.4 (GND); no longer C22.2, C23.1, C24.2, C27.2, R26.2
- net RF_AUDIO: now also R33.2; no longer C30.2, R28.2, R29.1
- net at R15.1: now also C27.2, R34.1; no longer J3.2
- new net: C30.2, R28.2, R29.1, R33.1
- new net: C27.1, J3.2
- new net VGND: C22.2, C23.1, C24.2, R26.2, R34.2
Other:
- moved on the sheet: C22, C23, C24, C25, C26, C29, C30, C31, J3, J4, R15, R21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

Commit message: BOM CHANGES
Parts:
- C27: value 0.1uF -> 22nF
- R15, R21: value 1k -> 2k
- R25: value 4k -> 9k
- R34: value 100k -> 2k
Connections:
- net VGND: now also C27.2; no longer R34.2
- net at C25.2, U5.1, U5.2 (-)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: now also R34.2; no longer C26.1
- net at C27.1: now also C26.1, R34.1; no longer J3.2
- new net: J3.2, R15.1
Other:
- moved on the sheet: C26, C27, R34

Commit message: saving
Connections:
- net at R26.1, U5.6 (-): now also R25.1; no longer R25.2
- net at C30.1, U5.7: now also R25.2; no longer R25.1
Other:
- moved on the sheet: R25
Changed lines of the file:
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@@
 	(symbol
 		(lib_id "Device:R")
-		(at 146.05 100.33 0)
+		(at 146.05 100.33 180)
 		(unit 1)
 		(exclude_from_sim no)
@@
 					(size 1.27 1.27)
 				)
-				(justify left)
+				(justify right)
 			)
 		)
@@
 					(size 1.27 1.27)
 				)
-				(justify left)
+				(justify right)
 			)
 		)
 		(property "Footprint" "Resistor_SMD:R_0402_1005Metric"
-			(at 144.272 100.33 90)
+			(at 147.828 100.33 90)
 			(effects
 				(font

Commit message: changed audio section
Parts:
- removed C22, C23: 47uF, Capacitor_SMD:C_0805_2012Metric, symbol Device:C
- removed C24, C25, C27: 22nF, Capacitor_SMD:C_0402_1005Metric, symbol Device:C
- removed C26: 1uF, Capacitor_SMD:C_0402_1005Metric, symbol Device:C
- removed C29: 0.05uF, Capacitor_SMD:C_0402_1005Metric, symbol Device:C
- removed C30: 0.1uF, Capacitor_SMD:C_0402_1005Metric, symbol Device:C
- removed C31: 200uF, Capacitor_SMD:CP_Elec_6.3x4.5, symbol Device:C
- removed J3: SJ-43514, Custom_footprints:CUI_SJ-43514, symbol SJ-43514:SJ-43514
- removed J4: SPEAKER_OUT, Connector_PinHeader_2.54mm:PinHeader_1x02_P2.54mm_Vertical, symbol Connector:Conn_01x02_Pin
- removed R15, R21, R34: 2k, Resistor_SMD:R_0402_1005Metric, symbol Device:R
- removed R25: 9k, Resistor_SMD:R_0402_1005Metric, symbol Device:R
- removed R26, R33: 1k, Resistor_SMD:R_0402_1005Metric, symbol Device:R
- removed R27: 10, Resistor_SMD:R_0402_1005Metric, symbol Device:R
- removed R28, R29: 100k, Resistor_SMD:R_0402_1005Metric, symbol Device:R
- removed U5: TL072, Package_DIP:DIP-8_W7.62mm, symbol Amplifier_Operational:TL072
- removed U6: LM386, Package_DIP:DIP-8_W7.62mm, symbol Amplifier_Audio:LM386
Connections:
- net GND: no longer J11.2 (Pin_2), J12.2 (Pin_2), J6.5 (Pin_5), J8.7 (Pin_7)
- new net SGND: J11.2 (Pin_2), J12.2 (Pin_2), J6.5 (Pin_5), J8.7 (Pin_7)
