File: Proton-KiCAD/Proton.kicad_pcb (KiCad board)
At the start: 4 copper layers, 20.3 x 99.1 mm, 119 parts, among them J1 USB_C_Receptacle_USB2.0_14P, J2 Conn_01x28_Pin, J3 DebugnBoot, J4 Conn_01x28_Pin, J5 USB_C_Receptacle_USB2.0_14P, J6 Conn_02x03_Top_Bottom, J7 UART-PINS, SW1 BOOTSEL, SW2 RESET, SW3 LEFT, SW4 RIGHT, U1 W25Q128JVS, U10 USBLC6-2P6, U2 NCP1117-3.3_SOT223, U3 RP2350_80QFN, U4 W25Q16JVUXIQ TR, U5 AP2112K-3.3, U6 RP2040, U7 SN74AUP1T17DCKR, U8 SN74AUP1T17DCKR, U9 USBLC6-2P6, Y1 ABM8-272-T3, Y2 ABM8-272-T3

Commit message: working on 4layer proton
Parts:
- removed C1, C2, C24, C25: 15p, Capacitor_SMD:C_0402_1005Metric
- removed C10, C9: 4.7u, Capacitor_SMD:C_0402_1005Metric
- removed C11, C13, C14, C15, C16, C17, C18, C19, C20, C21, C22, C23, C28, C29, C3, C30, C33, C35, C36, C37, C38, C39, C40, C41, C42, C8: 100n, Capacitor_SMD:C_0402_1005Metric
- removed C12, C26, C4, C7: 10u, Capacitor_SMD:C_0805_2012Metric
- removed C27, C32: 10u, Capacitor_SMD:C_0603_1608Metric
- removed C31, C34: 1u, Capacitor_SMD:C_0402_1005Metric
- removed C5, C6: 4.7u, RP2350_80QFN_minimal:C_0402_1005Metric_small_pads
- removed CR1, CR2: BAT60JFILM, BAT60JFILM:CR_60JFILM_STM
- removed D1: RED, Diode_SMD:D_0402_1005Metric
- removed D2, D4: GREEN, Diode_SMD:D_0402_1005Metric
- removed D3, D5: YELLOW, Diode_SMD:D_0402_1005Metric
- removed G***: LOGO, logos:purdue-small
- removed G*** (x3): LOGO, LOGO
- removed G***: LOGO, logos:362-small
- removed J1, J5: USB_C_Receptacle_USB2.0_14P, Connector_USB:USB_C_Receptacle_G-Switch_GT-USB-7010ASV
- removed J2, J4: Conn_01x28_Pin, Connector_PinHeader_2.54mm:PinHeader_1x28_P2.54mm_Vertical
- removed J3: DebugnBoot, Connector_PinHeader_2.54mm:PinHeader_1x04_P2.54mm_Vertical
- removed J6: Conn_02x03_Top_Bottom, Connector_PinSocket_2.54mm:PinSocket_2x03_P2.54mm_Vertical
- removed J7: UART-PINS, Connector_PinHeader_2.54mm:PinHeader_1x03_P2.54mm_Vertical
- removed L1: 3.3u, RP2350_80QFN_minimal:L_pol_2016
- removed PD1, UD1: RED, LED_SMD:LED_0805_2012Metric
- removed PD2, UD3: GREEN, LED_SMD:LED_0805_2012Metric
- removed R1, R18, R19, R2, R6: 5.1k, Resistor_SMD:R_0402_1005Metric
- removed R10, R21, R22, R9: 27, Resistor_SMD:R_0402_1005Metric
- removed R11: 3k, Resistor_SMD:R_0402_1005Metric
- removed R12, R14, R15, R17, R20, R3, R4, R7, R8: 1k, Resistor_SMD:R_0402_1005Metric
- removed R13, R30, R32: 2k, Resistor_SMD:R_0402_1005Metric
- removed R16: 510, Resistor_SMD:R_0402_1005Metric
- removed R23, R31, R33: 470, Resistor_SMD:R_0402_1005Metric
- removed R24, R25, R26, R27, R28, R29: 100, Resistor_SMD:R_0402_1005Metric
- removed R34, R35: 10k, Resistor_SMD:R_0402_1005Metric
- removed R5: 33, Resistor_SMD:R_0402_1005Metric
- removed SW1: BOOTSEL, Button_Switch_SMD:SW_SPST_PTS647_Sx38
- removed SW2: RESET, Button_Switch_SMD:SW_SPST_PTS647_Sx38
- removed SW3: LEFT, Button_Switch_SMD:SW_SPST_PTS647_Sx38
- removed SW4: RIGHT, Button_Switch_SMD:SW_SPST_PTS647_Sx38
- removed U1: W25Q128JVS, Package_SO:SOIC-8_5.23x5.23mm_P1.27mm
- removed U10, U9: USBLC6-2P6, Package_TO_SOT_SMD:SOT-666
- removed U2: NCP1117-3.3_SOT223, Package_TO_SOT_SMD:SOT-223-3_TabPin2
- removed U3: RP2350_80QFN, RP2350_80QFN_minimal:RP2350-QFN-80-1EP_10x10_P0.4mm_EP3.4x3.4mm_ThermalVias
- removed U4: W25Q16JVUXIQ TR, W25Q16JVUXIQ:USON-8_UX_2x3x0p6_WIN
- removed U5: AP2112K-3.3, Package_TO_SOT_SMD:SOT-23-5
- removed U6: RP2040, DebugProbe:RP2040-QFN-56
- removed U7, U8: SN74AUP1T17DCKR, SN74AUP1T17DCKR:DCK5
- removed UD2: YELLOW, LED_SMD:LED_0805_2012Metric
- removed UD4: BLUE, LED_SMD:LED_0805_2012Metric
- removed Y1, Y2: ABM8-272-T3, Crystal:Crystal_SMD_3225-4Pin_3.2x2.5mm
Routing:
- net +3V3: track 170.0 -> 0.00 mm, vias 11 -> 0
- net GND: track 80.1 -> 0.00 mm, vias 16 -> 0
- net +P3V3: track 65.9 -> 0.00 mm, vias 6 -> 0
- net PGND: track 60.4 -> 0.00 mm, vias 9 -> 0
- net VBUS: track 47.5 -> 0.00 mm
- net /GPIO24: track 41.1 -> 0.00 mm, vias 2 -> 0
- net /USB_D-: track 40.5 -> 0.00 mm, vias 2 -> 0
- net /USB_D+: track 40.4 -> 0.00 mm, vias 2 -> 0
- net /SWCLK: track 39.8 -> 0.00 mm, vias 1 -> 0
- net PSWD: track 39.4 -> 0.00 mm, vias 1 -> 0
- net /RUN: track 36.1 -> 0.00 mm, vias 2 -> 0
- net /SWD: track 36.1 -> 0.00 mm, vias 2 -> 0
- net /GPIO21: track 35.9 -> 0.00 mm, vias 1 -> 0
- net /GPIO26: track 35.3 -> 0.00 mm, vias 2 -> 0
- net /GPIO23: track 34.7 -> 0.00 mm, vias 2 -> 0
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- removed copper zone on F.Cu, net (none)
- removed copper zone on In1.Cu, net (none)
- removed copper zone on In2.Cu, net (none)
- removed copper zone on B.Cu, net GND
- removed copper zone on B.Cu, net PGND
Other:
- board outline removed
- board text removed: "0"
- board text removed: "1"
- board text removed: "10"
- board text removed: "11"
- board text removed: "12"
- board text removed: "13"
- board text removed: "14"
- board text removed: "15"
- board text removed: "16"
- board text removed: "17"
- board text removed: "18"
- board text removed: "19"
- board text removed: "2"
- board text removed: "20"
- board text removed: "21"
- board text removed: "22"
- board text removed: "23"
- board text removed: "24"
- board text removed: "25"
- board text removed: "26"
- board text removed: "27"
- board text removed: "28"
- board text removed: "29"
- board text removed: "3"
- board text removed: "30"
- board text removed: "31"
- board text removed: "32"
- board text removed: "33"
- board text removed: "34"
- board text removed: "35"
- board text removed: "36"
- board text removed: "37"
- board text removed: "38"
- board text removed: "39"
- board text removed: "3V3"
- board text removed: "4"
- board text removed: "40"
- board text removed: "41"
- board text removed: "42"
- board text removed: "43"
- board text removed: "44"
- board text removed: "45"
- board text removed: "46"
- board text removed: "47"
- board text removed: "5"
- board text removed: "5V"
- board text removed: "6"
- board text removed: "7"
- board text removed: "8"
- board text removed: "9"
- board text removed: "BOOTSEL"
- board text removed: "Blame Niraj!"
- board text removed: "Debug Probe for Purdue Proton Rev 2"
- board text removed: "GND"
- board text removed: "PBOOT"
- board text removed: "PGND"
- board text removed: "PSWCLK"
- board text removed: "PSWD"
- board text removed: "RESET"
- board text removed: "RP2350B Dev Board Rev 3"
- board text removed: "RX"
- board text removed: "SWCLK"
- board text removed: "SWD"
- board text removed: "TX"
- board text removed: "V-CUT"
- board text removed: "www.TechnologicalArts.com"

Commit message: did some layout
Parts:
- added C1: 15p, Capacitor_SMD:C_0402_1005Metric, F.Cu at (145.0, 73.8)
- added C10: 4.7u, Capacitor_SMD:C_0402_1005Metric, B.Cu at (157.9, 63.8)
- added C11: 100n, Capacitor_SMD:C_0402_1005Metric, B.Cu at (150.5, 67.3)
- added C12: 10u, Capacitor_SMD:C_0805_2012Metric, B.Cu at (157.9, 58.3)
- added C13: 100n, Capacitor_SMD:C_0402_1005Metric, B.Cu at (148.5, 56.8)
- added C14: 100n, Capacitor_SMD:C_0402_1005Metric, B.Cu at (152.0, 59.8)
- added C15: 100n, Capacitor_SMD:C_0402_1005Metric, B.Cu at (154.5, 60.9)
- added C16: 100n, Capacitor_SMD:C_0402_1005Metric, B.Cu at (153.9, 63.8)
- added C17: 100n, Capacitor_SMD:C_0402_1005Metric, B.Cu at (153.4, 67.3)
- added C18: 100n, Capacitor_SMD:C_0402_1005Metric, B.Cu at (147.5, 67.3)
- added C19: 100n, Capacitor_SMD:C_0402_1005Metric, B.Cu at (147.4, 63.8)
- added C2: 15p, Capacitor_SMD:C_0402_1005Metric, F.Cu at (151.0, 73.8)
- added C20: 100n, Capacitor_SMD:C_0402_1005Metric, B.Cu at (147.5, 61.3)
- added C21: 100n, Capacitor_SMD:C_0402_1005Metric, B.Cu at (147.4, 59.8)
- added C22: 15p, Capacitor_SMD:C_0402_1005Metric, F.Cu at (139.2, 60.5)
- added C23: 15p, Capacitor_SMD:C_0402_1005Metric, F.Cu at (130.7, 60.5)
- added C24: 10u, Capacitor_SMD:C_0805_2012Metric, F.Cu at (139.5, 39.8)
- added C25: 10u, Capacitor_SMD:C_0603_1608Metric, F.Cu at (144.5, 43.6)
- added C26: 100n, Capacitor_SMD:C_0402_1005Metric, F.Cu at (123.9, 43.3)
- added C27: 100n, Capacitor_SMD:C_0402_1005Metric, F.Cu at (29.6, 76.9)
- added C28: 100n, Capacitor_SMD:C_0402_1005Metric, F.Cu at (32.5, 71.0)
- added C29: 1u, Capacitor_SMD:C_0402_1005Metric, F.Cu at (32.5, 73.0)
- added C3: 100n, Capacitor_SMD:C_0402_1005Metric, F.Cu at (153.4, 47.8)
- added C30: 10u, Capacitor_SMD:C_0603_1608Metric, F.Cu at (16.8, 86.0)
- added C31: 100n, Capacitor_SMD:C_0402_1005Metric, F.Cu at (32.5, 74.9)
- added C32: 1u, Capacitor_SMD:C_0402_1005Metric, F.Cu at (32.5, 76.9)
- added C33: 100n, Capacitor_SMD:C_0402_1005Metric, F.Cu at (35.3, 71.0)
- added C34: 100n, Capacitor_SMD:C_0402_1005Metric, F.Cu at (35.3, 73.0)
- added C35: 100n, Capacitor_SMD:C_0402_1005Metric, F.Cu at (35.3, 74.9)
- added C36: 100n, Capacitor_SMD:C_0402_1005Metric, F.Cu at (35.3, 76.9)
- added C37: 100n, Capacitor_SMD:C_0402_1005Metric, F.Cu at (38.2, 71.0)
- added C38: 100n, Capacitor_SMD:C_0402_1005Metric, F.Cu at (38.2, 73.0)
- added C39: 100n, Capacitor_SMD:C_0402_1005Metric, F.Cu at (128.0, 52.5)
- added C4: 10u, Capacitor_SMD:C_0805_2012Metric, F.Cu at (159.0, 46.4)
- added C40: 100n, Capacitor_SMD:C_0402_1005Metric, F.Cu at (38.2, 76.9)
- added C41: 0.1uF, Capacitor_SMD:C_0402_1005Metric, F.Cu at (9.49, 69.3)
- added C42: 22nF, Capacitor_SMD:C_0402_1005Metric, F.Cu at (9.49, 71.2)
- added C43: 22nF, Capacitor_SMD:C_0402_1005Metric, F.Cu at (9.49, 73.2)
- added C44: 1uF, Capacitor_SMD:C_0402_1005Metric, F.Cu at (9.49, 75.2)
- added C45: 0.05, Capacitor_SMD:C_0402_1005Metric, F.Cu at (9.49, 77.1)
- added C46: 250uF, Capacitor_THT:CP_Radial_D10.0mm_P5.00mm, F.Cu at (-9.39, 74.1)
- added C47: 10uF, Capacitor_SMD:C_0805_2012Metric, F.Cu at (-15.3, 76.6)
- added C48: .1uF, Capacitor_SMD:C_0402_1005Metric, F.Cu at (9.49, 79.1)
- added C5: 4.7u, Capacitor_SMD:C_0402_1005Metric, B.Cu at (143.5, 61.9)
- added C6: 4.7u, Capacitor_SMD:C_0402_1005Metric, B.Cu at (143.5, 63.8)
- added C7: 10u, Capacitor_SMD:C_0805_2012Metric, F.Cu at (155.5, 50.4)
- added C8: 100n, Capacitor_SMD:C_0402_1005Metric, B.Cu at (157.9, 61.3)
- added C9: 4.7u, Capacitor_SMD:C_0402_1005Metric, B.Cu at (155.5, 56.8)
- added D1: RED, Diode_SMD:D_0402_1005Metric, F.Cu at (119.5, 38.3)
- added D2: GREEN, Diode_SMD:D_0402_1005Metric, F.Cu at (32.8, 84.9)
- added D3: YELLOW, Diode_SMD:D_0402_1005Metric, F.Cu at (32.8, 86.9)
- added D4: GREEN, Diode_SMD:D_0402_1005Metric, F.Cu at (118.9, 46.3)
- added D5: YELLOW, Diode_SMD:D_0402_1005Metric, F.Cu at (118.0, 43.3)
- added J1: USB_C_Receptacle_USB2.0_14P, Connector_USB:USB_C_Receptacle_G-Switch_GT-USB-7010ASV, F.Cu at (151.1, 39.8)
- added J10: OLED, Connector_PinHeader_2.54mm:PinHeader_1x14_P2.54mm_Vertical, F.Cu at (-24.4, 43.3)
- added J11: SI4703, Connector_PinHeader_2.54mm:PinHeader_1x08_P2.54mm_Vertical, F.Cu at (-15.2, 55.0)
- added J2: Conn_02x03_Top_Bottom, Connector_PinSocket_2.54mm:PinSocket_2x03_P2.54mm_Vertical, F.Cu at (19.7, 56.2)
- added J3: USB_C_Receptacle_USB2.0_14P, Connector_USB:USB_C_Receptacle_G-Switch_GT-USB-7010ASV, F.Cu at (131.0, 39.3)
- added J4: DebugnBoot, Connector_PinHeader_2.54mm:PinHeader_1x04_P2.54mm_Vertical, F.Cu at (17.1, 72.3)
- added J5: KEYPAD, Connector_PinHeader_2.54mm:PinHeader_1x08_P2.54mm_Vertical, F.Cu at (-19.8, 55.0)
- added J6: RF_OUTPUT, Connector_Audio:Jack_3.5mm_CUI_SJ1-3525N_Horizontal, F.Cu at (-5.54, 61.8)
- added J7: SPEAKER_OUT, Connector_PinHeader_2.54mm:PinHeader_1x02_P2.54mm_Vertical, F.Cu at (-19.8, 77.4)
- added J8: OLED SPI, Connector_PinHeader_2.54mm:PinHeader_1x04_P2.54mm_Vertical, F.Cu at (5.76, 70.6)
- added J9: ROTARY ENCODER, Connector_PinHeader_2.54mm:PinHeader_1x05_P2.54mm_Vertical, F.Cu at (1.17, 70.6)
- added PD1: RED, LED_SMD:LED_0805_2012Metric, F.Cu at (159.0, 42.3)
- added PD2: GREEN, LED_SMD:LED_0805_2012Metric, F.Cu at (162.5, 42.3)
- added R1: 5.1k, Resistor_SMD:R_0402_1005Metric, B.Cu at (152.5, 38.8)
- added R10: 27, Resistor_SMD:R_0402_1005Metric, F.Cu at (153.0, 56.4)
- added R11: 1k, Resistor_SMD:R_0402_1005Metric, F.Cu at (127.0, 48.3)
- added R12: 470, Resistor_SMD:R_0402_1005Metric, F.Cu at (119.4, 40.8)
- added R13: 5.1k, Resistor_SMD:R_0402_1005Metric, B.Cu at (131.9, 40.3)
- added R14: 5.1k, Resistor_SMD:R_0402_1005Metric, B.Cu at (129.9, 40.3)
- added R15: 1k, Resistor_SMD:R_0402_1005Metric, F.Cu at (132.2, 60.5)
- added R16: 27, Resistor_SMD:R_0402_1005Metric, F.Cu at (20.9, 81.0)
- added R17: 27, Resistor_SMD:R_0402_1005Metric, F.Cu at (23.8, 71.0)
- added R18: 100, Resistor_SMD:R_0402_1005Metric, F.Cu at (141.4, 52.8)
- added R19: 100, Resistor_SMD:R_0402_1005Metric, F.Cu at (141.4, 55.3)
- added R2: 5.1k, Resistor_SMD:R_0402_1005Metric, B.Cu at (149.0, 38.8)
- added R20: 100, Resistor_SMD:R_0402_1005Metric, F.Cu at (141.4, 57.8)
- added R21: 100, Resistor_SMD:R_0402_1005Metric, F.Cu at (23.8, 79.0)
- added R22: 100, Resistor_SMD:R_0402_1005Metric, F.Cu at (23.8, 81.0)
- added R23: 100, Resistor_SMD:R_0402_1005Metric, F.Cu at (26.7, 71.0)
- added R24: 2k, Resistor_SMD:R_0402_1005Metric, F.Cu at (26.7, 73.0)
- added R25: 470, Resistor_SMD:R_0402_1005Metric, F.Cu at (26.7, 75.0)
- added R26: 2k, Resistor_SMD:R_0402_1005Metric, F.Cu at (122.0, 46.3)
- added R27: 470, Resistor_SMD:R_0402_1005Metric, F.Cu at (121.0, 43.3)
- added R28: 1k, Resistor_SMD:R_0402_1005Metric, F.Cu at (2.64, 53.7)
- added R29: 1k, Resistor_SMD:R_0402_1005Metric, F.Cu at (2.64, 55.7)
- added R3: 1k, Resistor_SMD:R_0402_1005Metric, F.Cu at (151.0, 71.3)
- added R30: 1k, Resistor_SMD:R_0402_1005Metric, F.Cu at (2.64, 57.7)
- added R31: 1k, Resistor_SMD:R_0402_1005Metric, F.Cu at (2.64, 59.7)
- added R32: 1k, Resistor_SMD:R_0402_1005Metric, F.Cu at (2.64, 61.7)
- added R33: 1k, Resistor_SMD:R_0402_1005Metric, F.Cu at (2.64, 63.7)
- added R34: 100k, Resistor_SMD:R_0402_1005Metric, F.Cu at (2.64, 65.7)
- added R35: 50k, Resistor_SMD:R_0402_1005Metric, F.Cu at (5.55, 53.7)
- added R36: 1k, Resistor_SMD:R_0402_1005Metric, F.Cu at (5.55, 55.7)
- added R37: 10k, Resistor_SMD:R_0402_1005Metric, F.Cu at (5.55, 57.7)
- added R38: 1k, Resistor_SMD:R_0402_1005Metric, F.Cu at (5.55, 59.7)
- added R39: 10k, Resistor_SMD:R_0402_1005Metric, F.Cu at (5.55, 61.7)
- added R4: 1k, Resistor_SMD:R_0402_1005Metric, F.Cu at (168.0, 67.3)
- added R40: 1k, Resistor_SMD:R_0402_1005Metric, F.Cu at (5.55, 63.7)
- added R41: 1k, Resistor_SMD:R_0402_1005Metric, F.Cu at (5.55, 65.7)
- added R42: 10k, Resistor_SMD:R_0402_1005Metric, F.Cu at (8.46, 53.7)
- added R43: 10k, Resistor_SMD:R_0402_1005Metric, F.Cu at (8.46, 55.7)
- added R44: 4k, Resistor_SMD:R_0402_1005Metric, F.Cu at (8.46, 57.7)
- added R45: 1k, Resistor_SMD:R_0402_1005Metric, F.Cu at (8.46, 59.7)
- added R46: 4k, Resistor_SMD:R_0402_1005Metric, F.Cu at (8.46, 61.7)
- added R47: 1k, Resistor_SMD:R_0402_1005Metric, F.Cu at (8.46, 63.7)
- added R48: 100k, Resistor_SMD:R_0402_1005Metric, F.Cu at (8.46, 65.7)
- added R49: 100k, Resistor_SMD:R_0402_1005Metric, F.Cu at (11.4, 53.7)
- added R5: 33, Resistor_SMD:R_0402_1005Metric, B.Cu at (155.4, 54.3)
- added R50: 10, Resistor_SMD:R_0402_1005Metric, F.Cu at (11.4, 55.7)
- added R51: 10k, Resistor_SMD:R_0402_1005Metric, F.Cu at (11.4, 57.7)
- added R6: 1k, Resistor_SMD:R_0402_1005Metric, F.Cu at (168.0, 63.9)
- added R7: 5.1k, Resistor_SMD:R_0402_1005Metric, F.Cu at (159.0, 38.8)
- added R8: 1k, Resistor_SMD:R_0402_1005Metric, F.Cu at (162.5, 38.8)
- added R9: 27, Resistor_SMD:R_0402_1005Metric, F.Cu at (151.5, 56.4)
- added SW1: BOOTSEL, Button_Switch_SMD:SW_SPST_PTS647_Sx38, F.Cu at (163.5, 62.8)
- added SW2: RESET, Button_Switch_SMD:SW_SPST_PTS647_Sx38, F.Cu at (163.5, 69.3)
- added U1: W25Q128JVS, Package_SO:SOIC-8_5.3x5.3mm_P1.27mm, F.Cu at (148.0, 51.3)
- added U11: TL072, Package_DIP:DIP-8_W7.62mm, F.Cu at (-20.5, 43.1)
- added U12: LM386, Package_DIP:DIP-8_W7.62mm, F.Cu at (-9.75, 43.1)
- added U2: USBLC6-2P6, Package_TO_SOT_SMD:SOT-666, B.Cu at (151.1, 46.3)
- added U3: NCP1117-3.3_SOT223, Package_TO_SOT_SMD:SOT-223-3_TabPin2, F.Cu at (162.5, 53.4)
- added U4: RP2350_80QFN, Package_DFN_QFN:QFN-80-1EP_10x10mm_P0.4mm_EP3.4x3.4mm_ThermalVias, F.Cu at (150.5, 63.7)
- added U5: W25Q16JVUXIQ TR, Package_SON:Winbond_USON-8-1EP_3x2mm_P0.5mm_EP0.2x1.6mm, F.Cu at (123.0, 39.3)
- added U6: USBLC6-2P6, Package_TO_SOT_SMD:SOT-666, B.Cu at (131.0, 46.3)
- added U7: AP2112K-3.3, Package_TO_SOT_SMD:SOT-23-5, F.Cu at (139.4, 43.3)
- added U8: RP2040, Package_DFN_QFN:QFN-56-1EP_7x7mm_P0.4mm_EP3.2x3.2mm, F.Cu at (134.8, 54.1)
- added U9: SN74AUP1T17DCKR, Package_TO_SOT_SMD:Texas_R-PDSO-G5_DCK-5, F.Cu at (125.4, 53.5)
- added Y1: ABM8-272-T3, Crystal:Crystal_SMD_3225-4Pin_3.2x2.5mm, F.Cu at (147.9, 73.7)
- added Y2: ABM8-272-T3, Crystal:Crystal_SMD_3225-4Pin_3.2x2.5mm, F.Cu at (136.3, 60.6)
Other:
- board outline added: 61.5 x 57 mm

Commit message: working onlayout
Parts:
- removed C25: 10u, Capacitor_SMD:C_0603_1608Metric
- removed J2: Conn_02x03_Top_Bottom, Connector_PinSocket_2.54mm:PinSocket_2x03_P2.54mm_Vertical
- removed R46: 4k, Resistor_SMD:R_0402_1005Metric
- removed R47: 1k, Resistor_SMD:R_0402_1005Metric
- removed U7: AP2112K-3.3, Package_TO_SOT_SMD:SOT-23-5
- added R52: 4k, Resistor_SMD:R_0402_1005Metric, F.Cu at (197.2, 58.0)
- added R53: 1k, Resistor_SMD:R_0402_1005Metric, F.Cu at (197.3, 59.5)
- C24: value 10u -> 1uF; footprint Capacitor_SMD:C_0805_2012Metric -> Capacitor_SMD:C_0402_1005Metric
- C27, C28, C29, C31, C35, C36, C38, C4, C47, C48, C7, R10, R16, R17, R4, R6, R9: moved to B.Cu
- R35: value 50k -> 100k
- R44: value 4k -> 10k
- R45: value 1k -> 90k
- U6: moved to F.Cu
- moved J11 221.0 mm to (203.3, 87.5), turned to -90 degrees
- moved U11 207.1 mm to (186.2, 55.9)
- moved J8 201.9 mm to (207.5, 63.2)
- moved J7 201.1 mm to (177.8, 40.0), turned to 90 degrees
- moved J6 197.0 mm to (190.5, 42.2), turned to 180 degrees
- moved R51 193.9 mm to (205.0, 68.3), turned to 90 degrees
- moved R34 189.8 mm to (192.0, 52.2), turned to -90 degrees
- moved R44 188.8 mm to (197.2, 61.5)
- moved R45 188.8 mm to (197.2, 62.8), turned to 180 degrees
- moved R35 188.5 mm to (194.0, 52.2), turned to 90 degrees
- moved C46 188.4 mm to (176.8, 45.0), turned to -90 degrees
- moved R32 185.3 mm to (187.8, 52.3), turned to 90 degrees
- moved C43 182.2 mm to (190.5, 52.3), turned to -90 degrees
- moved U12 181.7 mm to (171.4, 55.9)
- moved R40 181.1 mm to (186.2, 52.3), turned to -90 degrees
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Connections:
- C24 pad 1: P_VBUS -> Net-(U11A--)
- C24 pad 2: GND -> Net-(U11B-+)
- C26 pad 1: +P3V3 -> +3.3V
- C30 pad 1: +P3V3 -> +3.3V
- C31 pad 1: +P3V3 -> +3.3V
- C32 pad 1: +P3V3 -> +3.3V
- C33 pad 1: +P3V3 -> +3.3V
- C34 pad 1: +P3V3 -> +3.3V
- C35 pad 1: +P3V3 -> +3.3V
- C36 pad 1: +P3V3 -> +3.3V
- C37 pad 1: +P3V3 -> +3.3V
- C38 pad 1: +P3V3 -> +3.3V
- C39 pad 1: +P3V3 -> +3.3V
- C40 pad 1: +P3V3 -> +3.3V
- C43 pad 2: RF_AUDIO -> Net-(U11A--)
- C44 pad 1: Net-(C44-Pad1) -> Net-(U11A--)
- R32 pad 2: Net-(R32-Pad2) -> Net-(C43-Pad1)
- R34 pad 1: Net-(C43-Pad1) -> +3.3V
- R40 pad 1: Net-(R32-Pad2) -> Net-(C43-Pad1)
- R44 pad 1: RF_AUDIO -> Net-(U11B-+)
- R44 pad 2: Net-(U11A--) -> GND
- R45 pad 1: Net-(U11A--) -> +3.3V
- R45 pad 2: GND -> Net-(U11B-+)
- U11 pad 1: RF_AUDIO -> Net-(U11A--)
- U11 pad 5: (no net) -> Net-(U11B-+)
- U11 pad 6: (no net) -> Net-(U11B--)
- U11 pad 7: (no net) -> RF_AUDIO
- U5 pad 8: +P3V3 -> +3.3V
- U8 pad 1: +P3V3 -> +3.3V
- U8 pad 10: +P3V3 -> +3.3V
- U8 pad 22: +P3V3 -> +3.3V
- U8 pad 33: +P3V3 -> +3.3V
- U8 pad 42: +P3V3 -> +3.3V
- U8 pad 43: +P3V3 -> +3.3V
- U8 pad 44: +P3V3 -> +3.3V
- U8 pad 48: +P3V3 -> +3.3V
- U8 pad 49: +P3V3 -> +3.3V
- U9 pad 5: +P3V3 -> +3.3V
Routing:
- net RF_~{RST}: track 0.00 -> 51.9 mm
- net RF_SCLK: track 0.00 -> 46.4 mm
- net RF_SDIO: track 0.00 -> 44.8 mm
- net RF_AUDIO: track 0.00 -> 39.5 mm, vias 0 -> 2
- net KEYPAD_GPIO2: track 0.00 -> 38.9 mm
- net ROT_SW: track 0.00 -> 27.9 mm, vias 0 -> 1
- net ROT_DT: track 0.00 -> 27.0 mm, vias 0 -> 2
- net ROT_CLK: track 0.00 -> 23.1 mm, vias 0 -> 1
- net Net-(U11B-+): track 0.00 -> 17.0 mm
- net Net-(U12-+): track 0.00 -> 16.5 mm
- net Net-(C46-Pad2): track 0.00 -> 14.5 mm
- net Net-(U11A--): track 0.00 -> 14.0 mm
- net Net-(U11A-+): track 0.00 -> 12.5 mm, vias 0 -> 1
- net Net-(C43-Pad1): track 0.00 -> 7.37 mm
- net /XIN: track 0.00 -> 6.60 mm
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- added copper zone on In2.Cu, net +3.3V
- added copper zone on B.Cu, net GND
- added copper zone on F.Cu, net GND
Other:
- board size 61.5 x 57 mm -> 92.6 x 57.2 mm

Commit message: Removing debugger
Parts:
- removed the C24 at (183.5, 61.0)
- removed the C26 at (137.2, 48.0)
- removed the C29 at (137.8, 51.5)
- removed the C31 at (132.5, 51.5)
- removed the C32 at (100.2, 50.5)
- removed the C33 at (138.8, 56.5)
- removed C34, C35, C36, C37, C38, C39, C40: 100n, Capacitor_SMD:C_0402_1005Metric
- removed C41: 0.1uF, Capacitor_SMD:C_0402_1005Metric
- removed D1: RED, Diode_SMD:D_0402_1005Metric
- removed D2, D4: GREEN, Diode_SMD:D_0402_1005Metric
- removed D3, D5: YELLOW, Diode_SMD:D_0402_1005Metric
- removed the J3 at (132.5, 40.3)
- removed the J4 at (84.8, 45.9)
- removed the R11 at (128.2, 49.2)
- removed the R12 at (139.5, 41.0)
- removed the R13 at (133.8, 42.2)
- removed the R14 at (130.8, 42.0)
- removed the R15 at (128.5, 56.8)
- removed the R16 at (133.8, 47.5)
- removed the R17 at (135.2, 47.5)
- removed the R18 at (128.2, 52.2)
- removed the R19 at (128.2, 53.9)
- removed the R20 at (128.2, 55.0)
- removed the R21 at (91.5, 52.5)
- removed the R22 at (91.5, 54.5)
- removed the R23 at (94.4, 44.5)
- removed the R24 at (94.4, 46.5)
- removed the R25 at (94.4, 48.5)
- removed the R26 at (141.0, 41.0)
- removed the R27 at (138.5, 41.0)
- removed R34, R35, R48, R49: 100k, Resistor_SMD:R_0402_1005Metric
- removed R44: 10k, Resistor_SMD:R_0402_1005Metric
- removed R45: 90k, Resistor_SMD:R_0402_1005Metric
- removed the U5 at (133.2, 46.8)
- removed the U6 at (129.5, 47.0)
- removed U8: RP2040, Package_DFN_QFN:QFN-56-1EP_7x7mm_P0.4mm_EP3.2x3.2mm
- removed U9: SN74AUP1T17DCKR, Package_TO_SOT_SMD:Texas_R-PDSO-G5_DCK-5
- removed Y2: ABM8-272-T3, Crystal:Crystal_SMD_3225-4Pin_3.2x2.5mm
- added CR1: BAT60JFILM, diode shite:CR_60JFILM_STM-M, B.Cu at (152.8, 46.5)
- added R28: 100k, Resistor_SMD:R_0402_1005Metric, F.Cu at (221.3, 74.0)
- added R29: 100k, Resistor_SMD:R_0402_1005Metric, F.Cu at (221.3, 76.0)
- C22, C23: value 15p -> 47uF; footprint Capacitor_SMD:C_0402_1005Metric -> Capacitor_SMD:C_0805_2012Metric
- C27, C28: value 100n -> 47uF; footprint Capacitor_SMD:C_0402_1005Metric -> Capacitor_SMD:C_0805_2012Metric; moved to F.Cu
- C30: value 10u -> 0.1uF; footprint Capacitor_SMD:C_0603_1608Metric -> Capacitor_SMD:C_0402_1005Metric
- moved C28 87.1 mm to (217.6, 77.5), turned to 0 degrees
- moved C30 86.2 mm to (221.3, 78.0), turned to 0 degrees
- moved C27 85.0 mm to (217.6, 74.5), turned to 0 degrees
- moved C22 63.4 mm to (197.2, 55.0), turned to 0 degrees
- moved C23 59.3 mm to (187.2, 67.0), turned to 180 degrees
- moved R4 47.5 mm to (104.0, 34.5), turned to -90 degrees
- moved R6 44.6 mm to (102.0, 41.0)
- moved SW1 44.6 mm to (103.0, 41.1)
- moved SW2 44.6 mm to (103.0, 35.5)
- moved C29 29.6 mm to (181.5, 69.5)
- moved R27 29.6 mm to (181.9, 71.7)
- moved R3 9.49 mm to (154.1, 74.6)
- moved C2 9.11 mm to (153.7, 76.4), turned to 180 degrees
- moved C10 7.59 mm to (148.2, 66.4)
- moved C11 7.59 mm to (148.2, 64.9)
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- renumbered C42 to C24, C43 to C25, C44 to C26, C45 to C29, C46 to C31, C47 to C32, C48 to C33, J5 to J2, J6 to J3, J7 to J4, J8 to J5, J9 to J6, J10 to J7, J11 to J8, R28 to R11, R29 to R12, R30 to R13, R31 to R14, R32 to R15, R33 to R16, R36 to R17, R37 to R18, R38 to R19, R39 to R20, R40 to R21, R41 to R22, R42 to R23, R43 to R24, R52 to R25, R53 to R26, R50 to R27, R51 to R30, U11 to U5, U12 to U6
Connections:
- C22 pad 1: /DebugProbe/XIN -> +3.3V
- C23 pad 1: Net-(C23-Pad1) -> GND
- C23 pad 2: GND -> Net-(U5C-V-)
- C25 pad 2: Net-(U11A--) -> Net-(U5A--)
- C26 pad 1: Net-(U11A--) -> Net-(U5A--)
- C27 pad 1: +P1V1 -> +5V
- C28 pad 1: +P1V1 -> Net-(U6-GND)
- C30 pad 1: +3.3V -> Net-(C30-Pad1)
- C30 pad 2: GND -> RF_AUDIO
- J3 pad TN: Net-(C41-Pad1) -> Net-(J3-PadTN)
- R15 pad 1: Net-(C41-Pad2) -> Net-(J3-PadTN)
- R25 pad 1: RF_AUDIO -> Net-(C30-Pad1)
- U5 pad 1: Net-(U11A--) -> Net-(U5A--)
- U5 pad 2: Net-(U11A--) -> Net-(U5A--)
- U5 pad 4: GND -> Net-(U5C-V-)
- U5 pad 5: Net-(U11B-+) -> Net-(U5A--)
- U5 pad 7: RF_AUDIO -> Net-(C30-Pad1)
- U6 pad 4: GND -> Net-(U6-GND)
Routing:
- net RF_~{RST}: track 51.9 -> 0.00 mm
- net RF_SCLK: track 46.4 -> 0.00 mm
- net RF_SDIO: track 44.8 -> 0.00 mm
- net RF_AUDIO: track 39.5 -> 0.00 mm, vias 2 -> 0
- net KEYPAD_GPIO2: track 38.9 -> 0.00 mm
- net ROT_SW: track 27.9 -> 0.00 mm, vias 1 -> 0
- net ROT_DT: track 27.0 -> 0.00 mm, vias 2 -> 0
- net ROT_CLK: track 23.1 -> 0.00 mm, vias 1 -> 0
- net Net-(U11B-+): track 17.0 -> 0.00 mm
- net Net-(U6-+): track 16.5 -> 0.00 mm
- net Net-(C31-Pad2): track 14.5 -> 0.00 mm
- net Net-(U11A--): track 14.0 -> 0.00 mm
- net Net-(U5A-+): track 12.5 -> 0.00 mm, vias 1 -> 0
- net Net-(C25-Pad1): track 7.37 -> 0.00 mm
- net /XIN: track 6.60 -> 0.00 mm
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