File: Proton-KiCAD/Proton.kicad_sch (KiCad schematic)
At the start: 62 parts, among them J1 USB_C_Receptacle_USB2.0_14P, J2 Conn_01x28_Pin, J4 Conn_01x28_Pin, J6 Conn_02x03_Top_Bottom, SW1 BOOTSEL, SW2 RESET, SW3 LEFT, SW4 RIGHT, U1 W25Q128JVS, U2 NCP1117-3.3_SOT223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

Commit message: working on 4layer proton
Parts:
- removed C22, C23: 100n, Capacitor_SMD:C_0402_1005Metric, symbol Device:C
- removed J2, J4: Conn_01x28_Pin, Connector_PinHeader_2.54mm:PinHeader_1x28_P2.54mm_Vertical, symbol Connector:Conn_01x28_Pin
- removed R11: 3k, Resistor_SMD:R_0402_1005Metric, symbol Device:R_US
- removed R12, R14, R15: 1k, Resistor_SMD:R_0402_1005Metric, symbol Device:R_US
- removed R13: 2k, Resistor_SMD:R_0402_1005Metric, symbol Device:R_US
- removed R16: 510, Resistor_SMD:R_0402_1005Metric, symbol Device:R_US
- removed R34, R35: 10k, Resistor_SMD:R_0402_1005Metric, symbol Device:R_US
- removed SW3: LEFT, Button_Switch_SMD:SW_SPST_PTS647_Sx38, symbol Switch:SW_Push
- removed SW4: RIGHT, Button_Switch_SMD:SW_SPST_PTS647_Sx38, symbol Switch:SW_Push
- removed UD1: RED, LED_SMD:LED_0805_2012Metric, symbol Device:LED
- removed UD2: YELLOW, LED_SMD:LED_0805_2012Metric, symbol Device:LED
- removed UD3: GREEN, LED_SMD:LED_0805_2012Metric, symbol Device:LED
- removed UD4: BLUE, LED_SMD:LED_0805_2012Metric, symbol Device:LED
Connections:
- net GPIO0 renamed UART_RX
- net GPIO1 renamed UART_TX
- net GPIO2 renamed KEYPAD_GPIO2
- net GPIO3 renamed KEYPAD_GPIO3
- net GPIO36 renamed RF_SDIO
- net GPIO37 renamed RF_SCLK
- net GPIO4 renamed KEYPAD_GPIO4
- net GPIO40_ADC0 renamed RF_~{RST}
- net GPIO5 renamed KEYPAD_GPIO5
- net GPIO6 renamed KEYPAD_GPIO6
- net GPIO7 renamed KEYPAD_GPIO7
- net GPIO8 renamed KEYPAD_GPIO8
- net GPIO9 renamed KEYPAD_GPIO9
Other:
- added sheet SSTV PERIPHERALS (untitled.kicad_sch)
- note removed: "IOs"
- note removed: "https://hackaday.com/2024/09/04/the-worsening-raspberry-pi-rp2350-e9-erratum-situation/"

Commit message: did some layout
Parts:
- C5, C6: footprint RP2350_80QFN_minimal:C_0402_1005Metric_small_pads -> Capacitor_SMD:C_0402_1005Metric
- U1: footprint Package_SO:SOIC-8_5.23x5.23mm_P1.27mm -> Package_SO:SOIC-8_5.3x5.3mm_P1.27mm
- U4: renamed from U3; footprint RP2350_80QFN_minimal:RP2350-QFN-80-1EP_10x10_P0.4mm_EP3.4x3.4mm_ThermalVias -> Package_DFN_QFN:QFN-80-1EP_10x10mm_P0.4mm_EP3.4x3.4mm_ThermalVias
- renumbered J6 to J2, R7 to R6, R6 to R7, U9 to U2, U2 to U3
Connections:
- net GPIO16 renamed OLED_SPI0_~{RST}
- net GPIO17 renamed OLED_SPI0_CS
- net GPIO18 renamed OLED_SPI0_SCLK
- net GPIO19 renamed OLED_SPI0_TX
- net GPIO20 renamed OLED_DC
- net GPIO27 renamed OLED_SPI1_TX
- net GPIO28 renamed OLED_SPI1_RX
- net GPIO29 renamed OLED_SPI1_CS
- net GPIO30 renamed OLED_SPI1_SCLK
- net GPIO32 renamed ROT_DT
- net GPIO33 renamed ROT_SW
- net GPIO34 renamed ROT_CLK
- net GPIO41_ADC1 renamed RF_AUDIO

Commit message: working onlayout
Parts:
- removed J2: Conn_02x03_Top_Bottom, Connector_PinSocket_2.54mm:PinSocket_2x03_P2.54mm_Vertical, symbol Connector_Generic:Conn_02x03_Top_Bottom
Changed lines of the file:
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@@
 	(wire
 		(pts
+			(xy 361.95 237.49) (xy 355.6 237.49)
+		)
+		(stroke
+			(width 0)
+			(type default)
+		)
+	)
+	(wire
+		(pts
 			(xy 217.17 95.25) (xy 217.17 107.95)
 		)
@@
 	(wire
 		(pts
-			(xy 368.3 232.41) (xy 384.81 232.41)
-		)
-		(stroke
-			(width 0)
-			(type default)
-		)
-	)
-	(wire
-		(pts
 			(xy 232.41 189.23) (xy 247.65 189.23)
 		)
@@
 	(wire
 		(pts
-			(xy 355.6 240.03) (xy 355.6 234.95)
+			(xy 355.6 240.03) (xy 355.6 237.49)
 		)
 		(stroke
@@
 		)
 	)
-	(wire
-		(pts
-			(xy 342.9 229.87) (xy 355.6 229.87)
-		)
-		(stroke
-			(width 0)
-			(type default)
-		)
-	)
 	(polyline
 		(pts
@@
 		)
 	)
-	(label "SWD"
-		(at 384.81 232.41 180)
-		(effects
-			(font
-				(size 1.27 1.27)
-			)
-			(justify right bottom)
-		)
-	)
 	(label "RUN"
 		(at 149.86 179.07 0)
@@
 		)
 	)
-	(label "SWCLK"
-		(at 342.9 229.87 0)
-		(effects
-			(font
-				(size 1.27 1.27)
-			)
-			(justify left bottom)
-		)
-	)
 	(label "GPIO30"
 		(at 247.65 201.93 180)
@@
 		)
 	)
-	(global_label "PSWD"
-		(shape input)
-		(at 368.3 234.95 0)
-		(fields_autoplaced yes)
-		(effects
-			(font
-				(size 1.27 1.27)
-			)
-			(justify left)
-		)
-		(property "Intersheetrefs" "${INTERSHEET_REFS}"
-			(at 375.8319 234.95 0)
-			(effects
-				(font
-					(size 1.27 1.27)
-				)
-				(justify left)
-				(hide yes)
-			)
-		)
-	)
 	(global_label "+5V"
 		(shape input)
@@
 		)
 	)
-	(global_label "PSWCLK"
-		(shape input)
-		(at 355.6 232.41 180)
-		(fields_autoplaced yes)
-		(effects
-			(font
-				(size 1.27 1.27)
-			)
-			(justify right)
-		)
-		(property "Intersheetrefs" "${INTERSHEET_REFS}"
-			(at 345.77 232.41 0)
-			(effects
-				(font
-					(size 1.27 1.27)
-				)
-				(justify right)
-				(hide yes)
-			)
-		)
-	)
 	(global_label "RF_SCLK"
 		(shape input)
@@
 	(global_label "PGND"
 		(shape input)
-		(at 368.3 229.87 0)
+		(at 361.95 237.49 0)
 		(fields_autoplaced yes)
 		(effects
@@
 		)
 		(property "Intersheetrefs" "${INTERSHEET_REFS}"
-			(at 375.7715 229.87 0)
+			(at 369.4215 237.49 0)
 			(effects
 				(font
@@
 					(unit 1)
 				)
-			)
-		)
-	)
-	(symbol
-		(lib_id "Connector_Generic:Conn_02x03_Top_Bottom")
-		(at 360.68 232.41 0)
-		(unit 1)
-		(exclude_from_sim no)
-		(in_bom yes)
-		(on_board yes)
-		(dnp no)
-		(fields_autoplaced yes)
-		(property "Reference" "J2"
-			(at 361.95 223.52 0)
-			(effects
-				(font
-					(size 1.27 1.27)
-				)
-				(hide yes)
-			)
-		)
-		(property "Value" "Conn_02x03_Top_Bottom"
-			(at 361.95 226.06 0)
-			(effects
-				(font
-					(size 1.27 1.27)
-				)
-				(hide yes)
-			)
-		)
-		(property "Footprint" "Connector_PinSocket_2.54mm:PinSocket_2x03_P2.54mm_Vertical"
-			(at 360.68 232.41 0)
-			(effects
-				(font
-					(size 1.27 1.27)
-				)
-				(hide yes)
-			)
-		)
-		(property "Datasheet" "~"
-			(at 360.68 232.41 0)
-			(effects
-				(font
-					(size 1.27 1.27)
-				)
-				(hide yes)
-			)
-		)
-		(property "Description" "Generic connector, double row, 02x03, top/bottom pin numbering scheme (row 1: 1...pins_per_row, row2: pins_per_row+1 ... num_pins), script generated (kicad-library-utils/schlib/autogen/connector/)"
-			(at 360.68 232.41 0)
-			(effects
-				(font
-					(size 1.27 1.27)
-				)
-				(hide yes)
-			)
-		)
-		(pin "1"
-		)
-		(pin "5"
-		)
-		(pin "3"
-		)
-		(pin "4"
-		)
-		(pin "6"
-		)
-		(pin "2"
-		)
-		(instances
-			(project ""
-				(path "/94683f5c-9cd9-448e-be96-9792537b5cb8"
-					(reference "J2")
-					(unit 1)
-				)

Commit message: Removing debugger
Parts:
- CR1: footprint BAT60JFILM:CR_60JFILM_STM -> diode shite:CR_60JFILM_STM-M
Other:
- removed sheet DebugProbe
Changed lines of the file:
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@@
 	(wire
 		(pts
-			(xy 361.95 237.49) (xy 355.6 237.49)
-		)
-		(stroke
-			(width 0)
-			(type default)
-		)
-	)
-	(wire
-		(pts
 			(xy 217.17 95.25) (xy 217.17 107.95)
 		)
@@
 	(wire
 		(pts
-			(xy 355.6 240.03) (xy 355.6 237.49)
-		)
-		(stroke
-			(width 0)
-			(type default)
-		)
-	)
-	(wire
-		(pts
 			(xy 152.4 83.82) (xy 152.4 85.09)
 		)
@@
 		)
 	)
-	(global_label "PGND"
-		(shape input)
-		(at 361.95 237.49 0)
-		(fields_autoplaced yes)
-		(effects
-			(font
-				(size 1.27 1.27)
-			)
-			(justify left)
-		)
-		(property "Intersheetrefs" "${INTERSHEET_REFS}"
-			(at 369.4215 237.49 0)
-			(effects
-				(font
-					(size 1.27 1.27)
-				)
-				(justify left)
-				(hide yes)
-			)
-		)
-	)
 	(global_label "OLED_SPI1_CS"
 		(shape input)
@@
 			)
 		)
-		(property "Footprint" "BAT60JFILM:CR_60JFILM_STM"
+		(property "Footprint" "diode shite:CR_60JFILM_STM-M"
 			(at 77.47 34.29 0)
 			(effects
@@
 	)
 	(symbol
-		(lib_name "GND_2")
-		(lib_id "power:GND")
-		(at 355.6 240.03 0)
-		(unit 1)
-		(exclude_from_sim no)
-		(in_bom yes)
-		(on_board yes)
-		(dnp no)
-		(fields_autoplaced yes)
-		(property "Reference" "#PWR034"
-			(at 355.6 246.38 0)
-			(effects
-				(font
-					(size 1.27 1.27)
-				)
-				(hide yes)
-			)
-		)
-		(property "Value" "GND"
-			(at 355.6 245.11 0)
-			(effects
-				(font
-					(size 1.27 1.27)
-				)
-			)
-		)
-		(property "Footprint" ""
-			(at 355.6 240.03 0)
-			(effects
-				(font
-					(size 1.27 1.27)
-				)
-				(hide yes)
-			)
-		)
-		(property "Datasheet" ""
-			(at 355.6 240.03 0)
-			(effects
-				(font
-					(size 1.27 1.27)
-				)
-				(hide yes)
-			)
-		)
-		(property "Description" "Power symbol creates a global label with name \"GND\" , ground"
-			(at 355.6 240.03 0)
-			(effects
-				(font
-					(size 1.27 1.27)
-				)
-				(hide yes)
-			)
-		)
-		(pin "1"
-		)
-		(instances
-			(project "RP2350_80QFN_minimal"
-				(path "/94683f5c-9cd9-448e-be96-9792537b5cb8"
-					(reference "#PWR034")
-					(unit 1)
-				)
-			)
-		)
-	)
-	(symbol
 		(lib_id "power:+3V3")
 		(at 105.41 101.6 0)
@@
 				)
 			)
-		)
-	)
-	(sheet
-		(at 36.83 119.38)
-		(size 35.56 21.59)
-		(exclude_from_sim no)
-		(in_bom yes)
-		(on_board yes)
-		(dnp no)
-		(fields_autoplaced yes)
-		(stroke
-			(width 0.1524)
-			(type solid)
-		)
-		(fill
-			(color 0 0 0 0.0000)
-		)
-		(property "Sheetname" "DebugProbe"
-			(at 36.83 118.6684 0)
-			(effects
-				(font
-					(size 1.27 1.27)
-				)
-				(justify left bottom)
-			)
-		)
-		(property "Sheetfile" "DebugProbe.kicad_sch"
-			(at 36.83 141.5546 0)
-			(effects
-				(font
-					(size 1.27 1.27)
-				)
-				(justify left top)
-			)
-		)
-		(instances
-			(project "Proton"
-				(path "/94683f5c-9cd9-448e-be96-9792537b5cb8"
-					(page "2")
-				)
-			)
