File: Proton-KiCAD/_autosave-Proton.kicad_pcb (KiCad board)
At the start: 4 copper layers, 92.6 x 57.2 mm, 85 parts, among them J1 USB_C_Receptacle_USB2.0_14P, J2 KEYPAD, J3 AudioJack3, J4 SPEAKER_OUT, J5 OLED SPI, J6 ROTARY ENCODER, J7 OLED, J8 SI4703, J9 Conn_01x03_Pin, SW1 BOOTSEL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

Commit message: need to spec audio jack
Parts:
- added H1: MountingHole, MountingHole:MountingHole_3.2mm_M3_DIN965_Pad, F.Cu at (206.7, 89.8)
- added H2: MountingHole, MountingHole:MountingHole_3.2mm_M3_DIN965_Pad, F.Cu at (124.3, 42.8)
- added H3: MountingHole, MountingHole:MountingHole_3.2mm_M3_DIN965_Pad, F.Cu at (206.7, 42.8)
- added H4: MountingHole, MountingHole:MountingHole_3.2mm_M3_DIN965_Pad, F.Cu at (124.3, 89.8)
- moved J3 5.30 mm to (195.0, 43.5)
- moved J4 3.54 mm to (183.5, 40.5)
Routing:
- net Net-(J4-Pin_1): track 6.58 -> 5.63 mm
