File: Proton-KiCAD/_autosave-Proton.kicad_sch (KiCad schematic)
At the start: 44 parts, among them J1 USB_C_Receptacle_USB2.0_14P, J9 Conn_01x03_Pin, SW1 BOOTSEL, SW2 RESET, U1 W25Q128JVS, U2 USBLC6-2P6, U3 NCP1117-3.3_SOT223, U4 RP2350_80QFN, Y1 ABM8-272-T3

Commit message: need to spec audio jack
Parts:
- added H1, H2, H3, H4: MountingHole, MountingHole:MountingHole_3.2mm_M3_DIN965_Pad, symbol Mechanical:MountingHole
Other:
- note removed: "Debugger Sheet (Link)"
