File: Proton-KiCAD2/DebugProbe.kicad_sch (KiCad schematic)
At the start: 47 parts, among them J3 USB_C_Receptacle_USB2.0_14P, J4 DebugnBoot, U10 SN74AUP1T17DCKR, U5 W25Q16JVUXIQ TR, U6 USBLC6-2P6, U8 RP2040, U9 SN74AUP1T17DCKR, Y2 ABM8-272-T3

Commit message: working onlayout
Parts:
- added C?: 10u, Capacitor_SMD:C_0603_1608Metric, symbol Device:C
- added C?: 10u, Capacitor_SMD:C_0805_2012Metric, symbol Device:C
- added CR?: BAT60JFILM, BAT60JFILM:CR_60JFILM_STM, symbol BAT60JFILM:BAT60JFILM
- added J?: UART-PINS, Connector_PinHeader_2.54mm:PinHeader_1x03_P2.54mm_Vertical, symbol Connector:Conn_01x03_Pin
- added U?: AP2112K-3.3, Package_TO_SOT_SMD:SOT-23-5, symbol Regulator_Linear:AP2112K-3.3
- U?: renamed from U8; footprint Package_DFN_QFN:QFN-56-1EP_7x7mm_P0.4mm_EP3.2x3.2mm -> DebugProbe:RP2040-QFN-56
- U?: renamed from U9; footprint Package_TO_SOT_SMD:Texas_R-PDSO-G5_DCK-5 -> SN74AUP1T17DCKR:DCK5
- U?: renamed from U5; footprint Package_SON:Winbond_USON-8-1EP_3x2mm_P0.5mm_EP0.2x1.6mm -> W25Q16JVUXIQ:USON-8_UX_2x3x0p6_WIN
- renumbered C38 to C?, C27 to C?, C28 to C?, C29 to C?, C32 to C?, C36 to C?, C37 to C?, C33 to C?, C40 to C?, C22 to C?, C35 to C?, C39 to C?, C30 to C?, C23 to C?, C34 to C?, C26 to C?, C31 to C?, D1 to D?, D4 to D?, D3 to D?, D2 to D?, D5 to D?, J4 to J3, J3 to J?, R24 to R?, R12 to R?, R21 to R?, R18 to R?, R22 to R?, R17 to R?, R25 to R?, R23 to R?, R13 to R?, R20 to R?, R14 to R?, R15 to R?, R27 to R?, R11 to R?, R19 to R?, R16 to R?, R26 to R?, U6 to U10, U10 to U?, Y2 to Y?
Connections:
- net +P3V3: now also C?.1, U?.5 (VOUT)
- net PGND: now also C?.2, C?.2, J?.2 (Pin_2), U?.2 (GND)
- net P_VBUS: now also C?.1, CR?.1, U?.1 (VIN), U?.3 (EN)
- net at J?.A4 (VBUS), J?.A9 (VBUS), J?.B4 (VBUS)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: now also CR?.2
- net UART_RX: no longer names the net of R?.2, R?.2
- net UART_RX: now also J?.3 (Pin_3)
- net UART_TX: no longer names the net of R?.2
- net UART_TX: now also J?.1 (Pin_1)
